File: Projects/Science Board/ScienceBoard-1.sch (KiCad schematic (older format))
At the start: 47 parts, among them J1 Stepper 1 In

Commit message: Add files via upload
Parts:
- removed J1: Stepper 1 In, symbol Connector_Generic:Conn_01x03
- removed J?: Conn_01x01, symbol Connector_Generic:Conn_01x01
- removed J?: Stepper 2 In, symbol Connector_Generic:Conn_01x03
- removed J?: Laser In, symbol Connector_Generic:Conn_01x02
- removed J?: Laser Out, symbol Connector_Generic:Conn_01x02
- removed J?: Motor 1 In, symbol Connector_Generic:Conn_01x03
- removed J?: Motor 2 Out, symbol Connector_Generic:Conn_01x03
- removed J?: From Arduino, symbol Connector_Generic:Conn_01x04
- removed J?: Conn_01x06, symbol Connector_Generic:Conn_01x06
- removed Q? (x6): Q_NPN_BCE, symbol Device:Q_NPN_BCE
- removed R? (x2): 1k, symbol Device:R
- removed R? (x2): 10k, symbol Device:R
- added J1: Conn_01x08, Connector_Molex:Molex_CLIK-Mate_502382-0870_1x08-1MP_P1.25mm_Vertical, symbol Connector_Generic:Conn_01x08
- added J2: Laser 1, MJ1-2533-SMT:CUI_MJ1-2533-SMT, symbol Connector_Generic:Conn_01x02
- added J5: Laser 2, MJ1-2533-SMT:CUI_MJ1-2533-SMT, symbol Connector_Generic:Conn_01x02
- added J6: 76825-0006, connector:Molex-76825-0006-0, symbol eec:76825-0006
- added R1, R2: 10k, Resistor_SMD:R_0402_1005Metric, symbol Device:R
- added R16: 4.3K, Resistor_SMD:R_0402_1005Metric, symbol Device:R_Small
- added R17: 100, Resistor_SMD:R_0402_1005Metric, symbol Device:R_Small
- added R18: 3K, Resistor_SMD:R_0402_1005Metric, symbol Device:R_Small
- added R19, R20, R21, R22, R23, R24: R_Small, Resistor_SMD:R_0402_1005Metric, symbol Device:R_Small
- added R5, R6: 1k, Resistor_SMD:R_0402_1005Metric, symbol Device:R
- added U5, U6, U7, U8: ZXTD09N50DE6, Package_TO_SOT_SMD:SOT-26, symbol Video:ZXTD09N50DE6
- added XA1: Arduino_Due_Shield, Arduino:Arduino_Due_Shield, symbol arduino:Arduino_Due_Shield
- C1, C2, C3, C4, C5, C6, C7: renamed from C?; footprint (none) -> Capacitor_SMD:C_0402_1005Metric
- J3, J4: renamed from J?; footprint (none) -> Connector_Molex:Molex_CLIK-Mate_502382-0470_1x04-1MP_P1.25mm_Vertical
- J8, J9: renamed from J?; footprint (none) -> Connector_Molex:Molex_CLIK-Mate_502382-0270_1x02-1MP_P1.25mm_Vertical
- L1: renamed from L?; footprint (none) -> Inductor_SMD:L_0402_1005Metric
- Q7: renamed from Q?; footprint (none) -> Package_TO_SOT_SMD:SOT-23
- R10, R12, R13, R15, R3, R4, R7, R8: renamed from R?; footprint (none) -> Resistor_SMD:R_0402_1005Metric
- R11: renamed from R?; value 243K -> 240K; footprint (none) -> Resistor_SMD:R_0402_1005Metric
- R14: renamed from R?; value 4.16 -> 4; footprint (none) -> Resistor_SMD:R_0402_1005Metric
- R9: renamed from R?; value 60.4K -> 56K; footprint (none) -> Resistor_SMD:R_0402_1005Metric
- U4: renamed from U?; footprint Package_SO:LTC_MSOP-16-1EP_3x4mm_P0.5mm_EP2.15x3.26mm -> Package_SO:MSOP-16-1EP_3x4mm_P0.5mm_EP1.65x2.85mm
- gave numbers to parts that had none: 3
Connections:
- net +24V: now also J6.4
- net 5V: now also R13.1, J1.4 (Pin_4), R1.1, R19.2, R2.1, R20.2; no longer R13.2
- net GND: now also J1.2 (Pin_2), J1.3 (Pin_3), J2.1 (Pin_1), J5.1 (Pin_1), J6.6, R17.2, R18.2, U5.2 (E1), U5.5 (E2), U6.2 (E1), U6.5 (E2), U7.2 (E1), U7.5 (E2), U8.2 (E1), U8.5 (E2); no longer R11.2, R9.2
- net ICG: now also J1.5 (Pin_5), XA1.D50
- net LASER1_CONTROL: now also R23.1, XA1.D13
- net LASER1_OUT: now also R10.1, J2.2 (Pin_2), U8.1 (C1)
- net LASER2_CONTROL: now also R24.2, XA1.D12
- net LASER2_OUT: now also R13.2, J5.2 (Pin_2), U8.3 (C2)
- net MOTOR1_CONTROL1: now also XA1.D5
- net MOTOR1_CONTROL2: now also XA1.D4 (D4_CS1)
- net MOTOR1_ENABLE: now also XA1.D32
- net MOTOR1_OUT1: now also J8.2 (Pin_2); no longer J8.1 (Pin_1)
- net MOTOR1_OUT2: now also J8.1 (Pin_1); no longer J8.2 (Pin_2)
- net MOTOR2_CONTROL1: now also XA1.D2
- net MOTOR2_CONTROL2: now also XA1.D3
- net MOTOR2_ENABLE: now also XA1.D30
- net MOTOR2_OUT1: now also J9.2 (Pin_2); no longer J9.1 (Pin_1)
- net MOTOR2_OUT2: now also J9.1 (Pin_1); no longer J9.2 (Pin_2)
- net OutputSignal_in: now also J1.8 (Pin_8)
- net OutputSignal_out: now also XA1.D44
- net SH: now also J1.6 (Pin_6), XA1.D48
- net STEPPER1_2A: now also R1.2, U5.3 (C2)
- net STEPPER1_3A: now also R2.2, U5.1 (C1)
- net STEPPER1_CONTROL1: now also R5.1, XA1.D6
- net STEPPER1_CONTROL2: now also R6.2, XA1.D7
- net STEPPER1_ENABLE: now also R19.1, U7.1 (C1)
- net STEPPER1_OUT1: now also J3.2 (Pin_2); no longer J3.4 (Pin_4)
- net STEPPER1_OUT2: now also J3.1 (Pin_1); no longer J3.3 (Pin_3)
- net STEPPER1_OUT3: now also J3.4 (Pin_4); no longer J3.2 (Pin_2), U1.14 (4Y)
- net STEPPER1_OUT4: now also J3.3 (Pin_3), U1.14 (4Y); no longer J3.1 (Pin_1)
- net STEPPER2_2A: now also U6.3 (C2)
- net STEPPER2_3A: now also U6.1 (C1)
- net STEPPER2_CONTROL1: now also R3.1, XA1.D9; no longer R3.2
- net STEPPER2_CONTROL2: now also XA1.D10 (D10_CS0)
- net STEPPER2_ENABLE: now also R20.1, U7.3 (C2)
- net STEPPER2_OUT1: now also J4.2 (Pin_2); no longer J4.4 (Pin_4)
- net STEPPER2_OUT2: now also J4.1 (Pin_1); no longer J4.3 (Pin_3)
- net STEPPER2_OUT3: now also J4.4 (Pin_4); no longer J4.2 (Pin_2)
- net STEPPER2_OUT4: now also J4.3 (Pin_3); no longer J4.1 (Pin_1)
- net SUCCESS_OUT: now also XA1.D52 (D52_CS2)
- net VPELT: now also J1.1 (Pin_1)
- net phiM(CCD_Clock): now also J1.7 (Pin_7), XA1.D46
- net at R4.1: now also U6.6 (B1)
- new net: R3.2, U6.4 (B2)
- new net: R16.1, R9.2
- new net: R11.2, R18.1
- new net: R24.1, U8.4 (B2)
- new net: R23.2, U8.6 (B1)
- new net: R16.2, R17.1
- new net: R5.2, U5.4 (B2)
- new net: R6.1, U5.6 (B1)
- new net: R22.1, U7.4 (B2)
- new net: R21.2, U7.6 (B1)
- new net STEPPER1_ENAB: R21.1, XA1.D38
- new net STEPPER2_ENAB: R22.2, XA1.D40
Other:
- moved on the sheet: C1, C5, C6, C7, J3, J4, L1, R10, R11, R12, R13, R14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
