File: Projects/ScienceBoard-2/ScienceBoard-1.kicad_pcb (KiCad board)
At the start: 4 copper layers, 128 x 53.6 mm, 80 parts, among them J1 Conn_01x08, J10 Conn_01x04, J2 Laser 1, J3 Conn_01x04, J4 Conn_01x02, J6 76825-0006, Q1 BTN8982TA, Q2 BTN8982TA, Q3 SUD50P04-08, Q7 Q_PNP_BCE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

Commit message: Add files via upload
Parts:
- added D7: MMSD4148, Diode_SMD:D_SOD-123, F.Cu at (83.1, 81.8)
- added F1: TR/3216FF25-R, Fuse:Fuse_1206_3216Metric, F.Cu at (96.3, 58.2)
- added K1: J115F11AH12VDCS61.5U, Relay_THT:Relay_StandexMeder_UMS, F.Cu at (80.4, 59.8)
- added Q4: TIP35CW, Package_TO_SOT_THT:TO-247-3_Vertical, F.Cu at (91.6, 90.9)
- moved J2 19.8 mm to (59.9, 49.5)
- moved J6 19.7 mm to (61.0, 85.3)
Connections:
- J6 pad 1: /12V -> /12V_in
- J6 pad 2: /12V -> /12V_in
- J6 pad 3: /12V -> /12V_in
- XA1 pad D14: Net-(XA1-PadD14) -> /ICG
- XA1 pad D19: /ICG -> Net-(XA1-PadD19)
- XA1 pad D51: Net-(XA1-PadD51) -> /POWER_ON
Routing:
- net /POWER_ON: track 0.00 -> 118.9 mm
- net /LASER1_OUT: track 19.6 -> 41.8 mm
- net Net-(D7-Pad2): track 0.00 -> 21.8 mm
- net /ICG: track 13.0 -> 18.4 mm, vias 0 -> 1
- net /STEPPER_LINE_OK: track 89.8 -> 89.2 mm
- net GND: track 76.1 -> 76.6 mm
- added copper zone on F.Cu, net /12V_in
- added copper zone on F.Cu, net Net-(F1-Pad2)
Other:
- board size 128 x 53.6 mm -> 147.8 x 53.6 mm

Commit message: Add files via upload
Parts:
- removed R16, R17: 0.2, Resistor_SMD:R_0402_1005Metric
- removed U8: ZXTD09N50DE6, Package_TO_SOT_SMD:SOT-26
- added D8: CMPD914E, Package_TO_SOT_SMD:SOT-23, F.Cu at (99.1, 44.5)
- added J5: Conn_01x02, Connector_Molex:Molex_KK-254_AE-6410-02A_1x02_P2.54mm_Vertical, F.Cu at (97.8, 49.8)
- added J7: Conn_01x02, Connector_Molex:Molex_KK-254_AE-6410-02A_1x02_P2.54mm_Vertical, F.Cu at (98.0, 64.5)
- added Q5: 2N7002, Package_TO_SOT_SMD:SOT-23, F.Cu at (104.9, 49.8)
- added Q6: SST4401, Package_TO_SOT_SMD:SOT-23, F.Cu at (109.7, 45.0)
- added Q8: NSS60201LT1G, Package_TO_SOT_SMD:SOT-23, F.Cu at (96.3, 71.6)
- added R13: 10k, Resistor_SMD:R_0402_1005Metric, B.Cu at (97.8, 92.5)
- C24: value 100uF -> 100nF
- C9: value 0.01uF -> 0.1uF
- R1: value 0.2 -> 8k
- R10: value 20 -> 5
- R2: value 0.2 -> 8
- R23: value R_Small -> 5k
- moved R2 76.4 mm to (98.6, 70.1)
- moved R1 73.0 mm to (98.6, 72.1), turned to 90 degrees
- moved R23 11.2 mm to (119.9, 46.0)
- moved R10 4.58 mm to (105.4, 42.4), turned to 180 degrees
- moved R22 1.85 mm to (102.4, 64.3), turned to 90 degrees
Connections:
- Q4 pad 1: /POWER_ON -> Net-(Q4-Pad1)
- R1 pad 1: Net-(R1-Pad1) -> Net-(Q8-Pad1)
- R1 pad 2: GND -> /LED_CONTROL
- R2 pad 1: Net-(R2-Pad1) -> /12V
- R2 pad 2: GND -> /LED_OUT
- U1 pad 5: Net-(R1-Pad1) -> GND
- U1 pad 8: Net-(R2-Pad1) -> GND
- U9 pad 5: Net-(R16-Pad1) -> GND
- U9 pad 8: Net-(R17-Pad1) -> GND
- XA1 pad D22: Net-(XA1-PadD22) -> /SOLENOID_ON
- XA1 pad D32: Net-(XA1-PadD32) -> /LED_CONTROL
Routing:
- net /LED_CONTROL: track 0.00 -> 99.9 mm, vias 0 -> 2
- net /SOLENOID_ON: track 0.00 -> 94.6 mm, vias 0 -> 5
- net GND: track 76.6 -> 98.2 mm, vias 89 -> 90
- net /LASER1_CONTROL: track 32.6 -> 21.4 mm
- net /LASER1_OUT: track 41.8 -> 52.2 mm
- net /SOLENOID_GND: track 0.00 -> 8.04 mm
- net /POWER_ON: track 118.9 -> 111.6 mm
- net Net-(Q4-Pad1): track 0.00 -> 6.38 mm
- net Net-(Q6-Pad1): track 2.72 -> 8.91 mm
- net /LED_OUT: track 0.00 -> 5.27 mm
- net Net-(R1-Pad1): track 4.81 -> 0.00 mm
- net Net-(R16-Pad1): track 4.80 -> 0.00 mm
- net /12V: track 0.00 -> 4.47 mm
- net Net-(R17-Pad1): track 3.98 -> 0.00 mm
- net Net-(R2-Pad1): track 3.48 -> 0.00 mm
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