File: Projects/ScienceBoard-2/ScienceBoard-1.kicad_pcb (KiCad board)
At the start: 4 copper layers, 147.8 x 53.6 mm, 88 parts, among them J1 Conn_01x08, J10 Conn_01x04, J2 Laser 1, J3 Conn_01x04, J4 Conn_01x02, J5 Conn_01x02, J6 76825-0006, J7 Conn_01x02, K1 J115F11AH12VDCS61.5U, Q1 BTN8982TA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

Commit message: Add files via upload
Parts:
- added C26: 4.7 uF, Capacitor_SMD:C_0402_1005Metric, F.Cu at (183.4, 53.4)
- added C27: 47 uF, Capacitor_SMD:C_0402_1005Metric, F.Cu at (184.7, 50.8)
- added R16: 3k, Resistor_SMD:R_0402_1005Metric, F.Cu at (184.7, 49.5)
- added R17: 20k, Resistor_SMD:R_0402_1005Metric, F.Cu at (106.9, 48.8)
- added R24: 20, Resistor_SMD:R_0402_1005Metric, F.Cu at (106.9, 51.6)
- added U3: NCP57302, Package_TO_SOT_SMD:TO-252-5_TabPin3, F.Cu at (177.0, 50.5)
- C12: value 0.01uF -> 0.1uF
- Q5: value 2N7002 -> FMMT634Q
- R14: value 4 -> 1k
- moved C7 10.7 mm to (167.1, 50.3)
- moved R15 8.24 mm to (164.3, 55.4), turned to 90 degrees
- moved Q7 7.18 mm to (166.9, 54.9), turned to 270 degrees
- moved Q5 4.58 mm to (109.4, 50.4), turned to 0 degrees
- moved R14 2.55 mm to (184.6, 48.3), turned to 180 degrees
- moved J1 2.54 mm to (188.7, 58.4)
Connections:
- C7 pad 1: GND -> /5V
- C7 pad 2: /5V -> GND
- Q5 pad 1: GND -> Net-(Q5-Pad1)
- Q5 pad 2: /SOLENOID_ON -> Net-(Q5-Pad2)
- Q5 pad 3: /SOLENOID_GND -> GND
- R14 pad 2: /5V -> Net-(R14-Pad2)
- XA1 pad A3: Net-(XA1-PadA3) -> /OutputSignal_out
- XA1 pad D10: Net-(XA1-PadD10) -> /SH
- XA1 pad D14: /ICG -> Net-(XA1-PadD14)
- XA1 pad D15: /OutputSignal_out -> Net-(XA1-PadD15)
- XA1 pad D16: /phiM(CCD_Clock) -> Net-(XA1-PadD16)
- XA1 pad D17: /SH -> Net-(XA1-PadD17)
- XA1 pad D2: Net-(XA1-PadD2) -> /phiM(CCD_Clock)
- XA1 pad D34: /OutputSignal_out -> Net-(XA1-PadD34)
- XA1 pad D9: Net-(XA1-PadD9) -> /ICG
Routing:
- net /SH: track 12.1 -> 53.2 mm, vias 0 -> 4
- net /ICG: track 18.4 -> 54.6 mm, vias 1 -> 2
- net /phiM(CCD_Clock): track 12.5 -> 23.2 mm, vias 0 -> 2
- net GND: track 98.2 -> 104.4 mm, vias 90 -> 96
- net Net-(R14-Pad2): track 0.00 -> 4.24 mm
- net /SOLENOID_GND: track 8.04 -> 12.1 mm
- net /5V: track 8.40 -> 11.6 mm
- net /OutputSignal_out: track 44.7 -> 42.3 mm, vias 1 -> 4
- net /BST2: track 25.9 -> 24.0 mm, vias 3 -> 4
- net Net-(Q5-Pad2): track 0.00 -> 1.61 mm
- net Net-(Q5-Pad1): track 0.00 -> 1.58 mm
- net /STEPPER2_OUT2: track 12.2 -> 13.3 mm, vias 1 -> 0
- net /STEPPER2_OUT1: track 11.9 -> 12.9 mm, vias 1 -> 0
- net /SOLENOID_ON: track 94.6 -> 93.7 mm
- net /STEPPER1_DIRECTION: track 7.34 -> 8.05 mm
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
Commit message: Add files via upload
Parts:
- removed C1: 0.1uF, Capacitor_SMD:C_0402_1005Metric
- removed C2, C3: 0.47 uF, Capacitor_SMD:C_0402_1005Metric
- removed C4, C5: 22uF, Capacitor_SMD:C_0402_1005Metric
- removed C6: 22uF, Capacitor_SMD:CP_Elec_4x5.8
- removed D3, D4: 12V, Diode_SMD:D_SMA
- removed D5, D6: 5V, Diode_SMD:D_SMA
- removed L1, L2: 4.3 uH, Inductor_SMD:L_Bourns-SRN6028
- removed R11, R30: 365, Resistor_SMD:R_0402_1005Metric
- removed R12, R18: 1.91k, Resistor_SMD:R_0402_1005Metric
- removed R9: 20k, Resistor_SMD:R_0402_1005Metric
- removed U2: LT3501, Package_SO:HTSSOP-20-1EP_4.4x6.5mm_P0.65mm_EP3.4x6.5mm_Mask2.75x3.43mm_ThermalVias
- added J8: Conn_01x06, Connector_Molex:Molex_KK-254_AE-6410-06A_1x06_P2.54mm_Vertical, F.Cu at (103.1, 76.2)
- moved Q8 1.02 mm to (97.3, 71.6)
- moved R1 1.02 mm to (99.6, 72.1)
- moved R2 1.02 mm to (99.6, 70.1)
Connections:
- C11 pad 1: /5V(Steppers) -> /5V
- C12 pad 1: /5V(Steppers) -> /5V
- C8 pad 1: /5V(Steppers) -> /5V
- C9 pad 1: /5V(Steppers) -> /5V
- R27 pad 2: /5V(Steppers) -> /5V
- R28 pad 1: /5V(Steppers) -> /5V
- R5 pad 2: /5V(Steppers) -> /5V
- R6 pad 1: /5V(Steppers) -> /5V
- U1 pad 17: /5V(Steppers) -> /5V
- U1 pad 18: /5V(Steppers) -> /5V
- U1 pad 19: /5V(Steppers) -> /5V
- U9 pad 17: /5V(Steppers) -> /5V
- U9 pad 18: /5V(Steppers) -> /5V
- U9 pad 19: /5V(Steppers) -> /5V
Routing:
- net /OTHER_LINE_OK: track 97.6 -> 0.00 mm, vias 1 -> 0
- net /STEPPER_LINE_OK: track 89.2 -> 0.00 mm, vias 1 -> 0
- net /REG_SHUTDOWN: track 67.7 -> 19.5 mm, vias 1 -> 0
- net /BST1: track 31.4 -> 0.00 mm, vias 3 -> 0
- net GND: track 104.4 -> 77.7 mm, vias 96 -> 87
- net /BST2: track 24.0 -> 0.00 mm, vias 4 -> 0
- net Net-(C3-Pad2): track 23.1 -> 0.00 mm
- net Net-(L2-Pad2): track 22.0 -> 0.00 mm
- net Net-(L1-Pad2): track 20.7 -> 0.00 mm, vias 2 -> 0
- net Net-(C2-Pad2): track 19.3 -> 0.00 mm, vias 2 -> 0
- net /5V(Steppers): track 17.6 -> 0.00 mm, vias 2 -> 0
- net /SOFT_START: track 14.9 -> 0.00 mm, vias 2 -> 0
- net /5V: track 11.6 -> 0.00 mm, vias 2 -> 0
- net /FB1: track 5.35 -> 0.00 mm
- net /FB2: track 5.30 -> 0.00 mm
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- removed copper zone on F.Cu, net /5V(Steppers)

Commit message: Add files via upload
Parts:
- added J11: Conn_01x02, Connector_Molex:Molex_KK-254_AE-6410-02A_1x02_P2.54mm_Vertical, F.Cu at (119.4, 73.4)
- added J9: Conn_01x02, Connector_Molex:Molex_KK-254_AE-6410-02A_1x02_P2.54mm_Vertical, F.Cu at (112.3, 73.4)
Connections:
- net /OTHER_LINE_OK renamed Net-(XA1-PadD53)
- net /REG_SHUTDOWN renamed Net-(XA1-PadD7)
- XA1 pad D10: /SH -> Net-(XA1-PadD10)
- XA1 pad D16: Net-(XA1-PadD16) -> /phiM(CCD_Clock)
- XA1 pad D2: /phiM(CCD_Clock) -> Net-(XA1-PadD2)
- XA1 pad D20: Net-(XA1-PadD20) -> /SH
- XA1 pad D21: Net-(XA1-PadD21) -> /ICG
- XA1 pad D34: Net-(XA1-PadD34) -> /LIMIT_SWITCH_1
- XA1 pad D52: /STEPPER_LINE_OK -> /LIMIT_SWITCH_2
- XA1 pad D9: /ICG -> Net-(XA1-PadD9)
Routing:
- net /LIMIT_SWITCH_1: track 0.00 -> 92.8 mm, vias 0 -> 2
- net /LIMIT_SWITCH_2: track 0.00 -> 84.3 mm, vias 0 -> 5
- net /ICG: track 54.6 -> 17.4 mm, vias 2 -> 0
- net /SH: track 53.2 -> 17.6 mm, vias 4 -> 0
- net /phiM(CCD_Clock): track 23.2 -> 16.5 mm, vias 2 -> 0
- net /OutputSignal_out: track 42.3 -> 43.0 mm, vias 4 -> 3

Commit message: Add files via upload
Parts:
- removed C26: 4.7 uF, Capacitor_SMD:C_0402_1005Metric
- removed C27: 47 uF, Capacitor_SMD:C_0402_1005Metric
- removed C7: 10 uF, Capacitor_SMD:CP_Elec_3x5.3
- removed Q7: Q_PNP_BCE, Package_TO_SOT_SMD:SOT-23
- removed Q8: NSS60201LT1G, Package_TO_SOT_SMD:SOT-23
- removed R14: 1k, Resistor_SMD:R_0402_1005Metric
- removed R15: 2.2k, Resistor_SMD:R_0402_1005Metric
- removed R16: 3k, Resistor_SMD:R_0402_1005Metric
- removed XA1: Arduino_Due_Shield, Arduino:Arduino_Due_Shield
- added R9: 5.1k, Resistor_SMD:R_0402_1005Metric, B.Cu at (167.9, 50.0)
- added U2: VO14642AT, Package_DIP:VO14642AT, F.Cu at (177.3, 58.4)
- added XA2: Arduino_Mega2560_Shield, Arduino:Arduino_Mega2560_Shield, F.Cu at (99.3, 94.8)
- Q6: value SST4401 -> FMMT634Q
- R1: value 8k -> 5.1k
- R23: moved to B.Cu
- U3: value NCP57302 -> VO14642AT; footprint Package_TO_SOT_SMD:TO-252-5_TabPin3 -> Package_DIP:VO14642AT
- moved U3 63.7 mm to (122.2, 83.1)
- moved R23 55.9 mm to (64.8, 55.4)
- moved Q6 50.6 mm to (60.5, 56.4), turned to 270 degrees
- moved R1 33.1 mm to (129.8, 85.6), turned to 0 degrees
- moved R2 21.8 mm to (114.3, 86.1), turned to 0 degrees
- moved J7 21.1 mm to (111.8, 80.5)
- moved J1 8.13 mm to (188.7, 50.3)
- moved R10 3.89 mm to (109.2, 43.2), turned to 0 degrees
Connections:
- J1 pad 4: /5V -> /OutputSignal_out
- J1 pad 8: /OutputSignal_in -> /VCCD
- J2 pad 1: GND -> /LASER1_GND
- Q6 pad 2: /LASER1_OUT -> /LASER1_GND
- R1 pad 1: Net-(Q8-Pad1) -> Net-(R1-Pad1)
- U3 pad 1: /5V -> Net-(R1-Pad1)
- U3 pad 2: /5V -> GND
- U3 pad 3: GND -> Net-(U3-Pad3)
- U3 pad 4: /VPELT -> GND
Routing:
- net /LASER1_CONTROL: track 21.4 -> 80.4 mm, vias 1 -> 0
- net /LED_CONTROL: track 98.8 -> 58.2 mm, vias 1 -> 8
- net Net-(XA2-PadD7): track 0.00 -> 19.5 mm
- net Net-(XA1-PadD7): track 19.5 -> 0.00 mm
- net /12V: track 4.47 -> 22.2 mm
- net /OutputSignal_out: track 43.0 -> 60.1 mm, vias 3 -> 2
- net /VPELT: track 0.00 -> 14.0 mm
- net Net-(R9-Pad1): track 0.00 -> 9.16 mm, vias 0 -> 1
- net /SH: track 17.6 -> 10.1 mm
- net GND: track 77.7 -> 70.3 mm, vias 87 -> 78
- net /ICG: track 17.4 -> 10.6 mm
- net /OutputSignal_in: track 6.54 -> 0.00 mm
- net Net-(Q6-Pad1): track 8.91 -> 2.89 mm, vias 0 -> 1
- net /LASER1_OUT: track 52.2 -> 46.3 mm
- net /PELTIER_ON: track 0.00 -> 5.59 mm, vias 0 -> 2
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- removed copper zone on F.Cu, net /VPELT
Other:
- board size 147.8 x 53.6 mm -> 147.8 x 53.3 mm

Commit message: Add files via upload
Parts:
- J6: value 76825-0006 -> Conn_01x02; footprint connector:Molex-76825-0006-0 -> Connector_Molex:Molex_Mega-Fit_76829-0002_2x01_P5.70mm_Vertical
- J8: footprint Connector_Molex:Molex_KK-254_AE-6410-06A_1x06_P2.54mm_Vertical -> Connector_Molex:Molex_Micro-Fit_3.0_43045-0612_2x03_P3.00mm_Vertical
- moved J8 12.5 mm to (91.4, 80.8)
- moved Q4 10.8 mm to (80.8, 90.7)
- moved R2 10.3 mm to (107.4, 78.5), turned to 270 degrees
- moved D7 9.32 mm to (74.2, 79.0)
- moved R13 4.62 mm to (93.2, 91.9), turned to 180 degrees
- moved J6 3.06 mm to (57.9, 85.1), turned to 90 degrees
Connections:
- J6 pad 1: /12V_in -> GND
- J8 pad 2: /12V -> GND
- J8 pad 3: GND -> /5V
- J8 pad 4: GND -> /12V
- J8 pad 5: /5V -> GND
Routing:
- net /12V: track 22.2 -> 0.00 mm
- net /POWER_ON: track 111.6 -> 121.0 mm
- net /LED_OUT: track 7.13 -> 16.2 mm
- net Net-(Q4-Pad1): track 6.38 -> 12.5 mm
- net Net-(D7-Pad2): track 21.8 -> 16.3 mm
- net (no net): vias 0 -> 4

Commit message: Add files via upload
Parts:
- removed R10: 5, Resistor_SMD:R_0402_1005Metric
- removed R23: 5k, Resistor_SMD:R_0402_1005Metric
- added R11: 5, Resistor_SMD:R_0402_1005Metric, F.Cu at (116.3, 47.5)
- added U6: LM317_3PinPackage, Package_TO_SOT_SMD:SOT-223-3_TabPin2, F.Cu at (121.7, 49.4)
- moved D2 6.43 mm to (127.8, 55.1)
- moved J2 0.25 mm to (60.2, 49.5)
- moved Q6 0.25 mm to (60.5, 56.1)
Connections:
- J1 pad 8: /VCCD -> /5V
- Q6 pad 1: Net-(Q6-Pad1) -> /LASER1_CONTROL
Routing:
- net Net-(XA2-PadD7): track 19.5 -> 0.00 mm
- net /LASER1_OUT: track 46.3 -> 57.6 mm
- net Net-(R11-Pad2): track 0.00 -> 3.78 mm
- net /LASER1_CONTROL: track 80.4 -> 84.2 mm, vias 0 -> 1
- net /POWER_ON: track 121.0 -> 117.7 mm
- net Net-(Q6-Pad1): track 2.89 -> 0.00 mm, vias 1 -> 0
- net /SOLENOID_ON: track 93.7 -> 96.0 mm, vias 5 -> 3
- net /LASER1_GND: track 4.24 -> 3.40 mm
- net /OutputSignal_out: track 60.1 -> 60.6 mm, vias 2 -> 0
- added copper zone on F.Cu, net Net-(R11-Pad2)
