File: Projects/ScienceBoard-2/ScienceBoard-1.sch (KiCad schematic (older format))
At the start: 80 parts, among them J1 Conn_01x08, J10 Conn_01x04, J2 Laser 1, J3 Conn_01x04, J4 Conn_01x02, J6 76825-0006, Q1 BTN8982TA, Q2 BTN8982TA, Q3 SUD50P04-08, Q7 Q_PNP_BCE, U1 DRV8834, U2 LT3501, U8 ZXTD09N50DE6, U9 DRV8834

Commit message: Add files via upload
Parts:
- added D7: MMSD4148, Diode_SMD:D_SOD-123, symbol Device:D
- added F1: TR/3216FF25-R, Fuse:Fuse_1206_3216Metric, symbol Device:Fuse
- added K1: J115F11AH12VDCS61.5U, Relay_THT:Relay_StandexMeder_UMS, symbol Relay:UMS05-1A80-75L
- added Q4: TIP35CW, Package_TO_SOT_THT:TO-247-3_Vertical, symbol Device:Q_NPN_BCE
Connections:
- net labels added: 12V_in, POWER_ON
- wire segments 160 -> 170
Other:
- moved on the sheet: J6
Changed lines of the file:
@@
 Text Label 14450 5550 0    50   ~ 0
 SH
-Text Label 14450 5750 0    50   ~ 0
+Text Label 14450 5250 0    50   ~ 0
 ICG
 $Comp
@@
 L eec:76825-0006 J6
 U 1 1 5FE0E70D
-P 6450 8750
-F 0 "J6" H 6208 9115 50  0000 C CNN
-F 1 "76825-0006" H 6208 9024 50  0000 C CNN
-F 2 "connector:Molex-76825-0006-0" H 6450 9250 50  0001 L CNN
-F 3 "https://www.molex.com/pdm_docs/sd/768250006_sd.pdf" H 6450 9350 50  0001 L CNN
-F 4 "Conn" H 6450 9450 50  0001 L CNN "category"
-F 5 "DUAL ROW RA HEADER TIN 6CKT" H 6450 9550 50  0001 L CNN "digikey description"
-F 6 "WM11971-ND" H 6450 9650 50  0001 L CNN "digikey part number"
-F 7 "yes" H 6450 9750 50  0001 L CNN "is connector"
-F 8 "yes" H 6450 9850 50  0001 L CNN "is male"
-F 9 "yes" H 6450 9950 50  0001 L CNN "lead free"
-F 10 "dc1b81f16b5cdc84" H 6450 10050 50  0001 L CNN "library id"
-F 11 "Molex" H 6450 10150 50  0001 L CNN "manufacturer"
-F 12 "538-76825-0006" H 6450 10250 50  0001 L CNN "mouser part number"
-F 13 "HDR6" H 6450 10350 50  0001 L CNN "package"
-F 14 "yes" H 6450 10450 50  0001 L CNN "rohs"
-F 15 "+105°C" H 6450 10550 50  0001 L CNN "temperature range high"
-F 16 "-40°C" H 6450 10650 50  0001 L CNN "temperature range low"
-	1    6450 8750
-	1    0    0    -1
-$EndComp
-Text Label 6350 8750 0    50   ~ 0
-12V
+P 6500 1150
+F 0 "J6" H 6258 1515 50  0000 C CNN
+F 1 "76825-0006" H 6258 1424 50  0000 C CNN
+F 2 "connector:Molex-76825-0006-0" H 6500 1650 50  0001 L CNN
+F 3 "https://www.molex.com/pdm_docs/sd/768250006_sd.pdf" H 6500 1750 50  0001 L CNN
+F 4 "Conn" H 6500 1850 50  0001 L CNN "category"
+F 5 "DUAL ROW RA HEADER TIN 6CKT" H 6500 1950 50  0001 L CNN "digikey description"
+F 6 "WM11971-ND" H 6500 2050 50  0001 L CNN "digikey part number"
+F 7 "yes" H 6500 2150 50  0001 L CNN "is connector"
+F 8 "yes" H 6500 2250 50  0001 L CNN "is male"
+F 9 "yes" H 6500 2350 50  0001 L CNN "lead free"
+F 10 "dc1b81f16b5cdc84" H 6500 2450 50  0001 L CNN "library id"
+F 11 "Molex" H 6500 2550 50  0001 L CNN "manufacturer"
+F 12 "538-76825-0006" H 6500 2650 50  0001 L CNN "mouser part number"
+F 13 "HDR6" H 6500 2750 50  0001 L CNN "package"
+F 14 "yes" H 6500 2850 50  0001 L CNN "rohs"
+F 15 "+105°C" H 6500 2950 50  0001 L CNN "temperature range high"
+F 16 "-40°C" H 6500 3050 50  0001 L CNN "temperature range low"
+	1    6500 1150
+	1    0    0    -1
+$EndComp
+Text Label 6400 1150 0    50   ~ 0
+12V_in
 $Comp
 L power:GND #PWR0127
 U 1 1 5FE0FF44
-P 6350 9750
-F 0 "#PWR0127" H 6350 9500 50  0001 C CNN
-F 1 "GND" V 6355 9577 50  0000 C CNN
-F 2 "" H 6350 9750 50  0001 C CNN
-F 3 "" H 6350 9750 50  0001 C CNN
-	1    6350 9750
+P 6400 2150
+F 0 "#PWR0127" H 6400 1900 50  0001 C CNN
+F 1 "GND" V 6405 1977 50  0000 C CNN
+F 2 "" H 6400 2150 50  0001 C CNN
+F 3 "" H 6400 2150 50  0001 C CNN
+	1    6400 2150
 	0    -1   -1   0
 $EndComp
-Text Label 6350 8950 0    50   ~ 0
-12V
-Text Label 6350 9150 0    50   ~ 0
-12V
+Text Label 6400 1350 0    50   ~ 0
+12V_in
+Text Label 6400 1550 0    50   ~ 0
+12V_in
 $Comp
 L power:GND #PWR0128
 U 1 1 5FFCB6FA
-P 6350 9350
-F 0 "#PWR0128" H 6350 9100 50  0001 C CNN
-F 1 "GND" V 6355 9222 50  0000 R CNN
-F 2 "" H 6350 9350 50  0001 C CNN
-F 3 "" H 6350 9350 50  0001 C CNN
-	1    6350 9350
+P 6400 1750
+F 0 "#PWR0128" H 6400 1500 50  0001 C CNN
+F 1 "GND" V 6405 1622 50  0000 R CNN
+F 2 "" H 6400 1750 50  0001 C CNN
+F 3 "" H 6400 1750 50  0001 C CNN
+	1    6400 1750
 	0    -1   -1   0
 $EndComp
@@
 L power:GND #PWR0129
 U 1 1 5FFCC514
-P 6350 9550
-F 0 "#PWR0129" H 6350 9300 50  0001 C CNN
-F 1 "GND" V 6355 9422 50  0000 R CNN
-F 2 "" H 6350 9550 50  0001 C CNN
-F 3 "" H 6350 9550 50  0001 C CNN
-	1    6350 9550
+P 6400 1950
+F 0 "#PWR0129" H 6400 1700 50  0001 C CNN
+F 1 "GND" V 6405 1822 50  0000 R CNN
+F 2 "" H 6400 1950 50  0001 C CNN
+F 3 "" H 6400 1950 50  0001 C CNN
+	1    6400 1950
 	0    -1   -1   0
 $EndComp
@@
 Text Label 14450 5350 0    50   ~ 0
 OutputSignal_out
+$Comp
+L Relay:UMS05-1A80-75L K1
+U 1 1 6052945E
+P 7750 1100
+F 0 "K1" V 8167 1100 50  0000 C CNN
+F 1 "J115F11AH12VDCS61.5U" V 8076 1100 50  0000 C CNN
+F 2 "Relay_THT:Relay_StandexMeder_UMS" H 8050 1050 50  0001 L CNN
+F 3 "https://standexelectronics.com/de/produkte/ums-reed-relais/" H 7750 1100 50  0001 C CNN
+	1    7750 1100
+	0    -1   -1   0
+$EndComp
+$Comp
+L Device:D D7
+U 1 1 6052B831
+P 7750 1850
+F 0 "D7" H 7750 2066 50  0000 C CNN
+F 1 "MMSD4148" H 7750 1975 50  0000 C CNN
+F 2 "Diode_SMD:D_SOD-123" H 7750 1850 50  0001 C CNN
+F 3 "~" H 7750 1850 50  0001 C CNN
+	1    7750 1850
+	1    0    0    -1
+$EndComp
+$Comp
+L Device:Q_NPN_BCE Q4
+U 1 1 6052C9F7
+P 8200 2200
+F 0 "Q4" H 8390 2246 50  0000 L CNN
+F 1 "TIP35CW" H 8390 2155 50  0000 L CNN
+F 2 "Package_TO_SOT_THT:TO-247-3_Vertical" H 8400 2300 50  0001 C CNN
+F 3 "~" H 8200 2200 50  0001 C CNN
+	1    8200 2200
+	1    0    0    -1
+$EndComp
+Wire Wire Line
+	7600 1850 7200 1850
+Wire Wire Line
+	7200 1850 7200 1300
+Wire Wire Line
+	7200 1300 7450 1300
+Wire Wire Line
+	8050 1300 8300 1300
+Wire Wire Line
+	8300 1300 8300 1850
+Wire Wire Line
+	7900 1850 8300 1850
+Connection ~ 8300 1850
+Wire Wire Line
+	8300 1850 8300 2000
+$Comp
+L power:GND #PWR0124
+U 1 1 6054B7FA
+P 8300 2400
+F 0 "#PWR0124" H 8300 2150 50  0001 C CNN
+F 1 "GND" H 8305 2227 50  0000 C CNN
+F 2 "" H 8300 2400 50  0001 C CNN
+F 3 "" H 8300 2400 50  0001 C CNN
+	1    8300 2400
+	1    0    0    -1
+$EndComp
+Text Label 8000 2200 2    50   ~ 0
+POWER_ON
+Wire Wire Line
+	7200 1300 7200 900
+Wire Wire Line
+	7200 900  7450 900
+Connection ~ 7200 1300
+$Comp
+L Device:Fuse F1
+U 1 1 6055518B
+P 8600 900
+F 0 "F1" V 8403 900 50  0000 C CNN
+F 1 "TR/3216FF25-R" V 8494 900 50  0000 C CNN
+F 2 "Fuse:Fuse_1206_3216Metric" V 8530 900 50  0001 C CNN
+F 3 "~" H 8600 900 50  0001 C CNN
+	1    8600 900
+	0    1    1    0
+$EndComp
+Text Label 8750 900  0    50   ~ 0
+12V
+Text Label 7200 1300 2    50   ~ 0
+12V_in
+Wire Wire Line
+	8050 900  8450 900
+Text Label 11850 1850 2    50   ~ 0
+POWER_ON
 $EndSCHEMATC

Commit message: Add files via upload
Parts:
- removed R1, R16, R17, R2: 0.2, Resistor_SMD:R_0402_1005Metric, symbol Device:R_Small
- removed U8: ZXTD09N50DE6, Package_TO_SOT_SMD:SOT-26, symbol Video:ZXTD09N50DE6
- added D8: CMPD914E, Package_TO_SOT_SMD:SOT-23, symbol Device:D
- added J5, J7: Conn_01x02, Connector_Molex:Molex_KK-254_AE-6410-02A_1x02_P2.54mm_Vertical, symbol Connector_Generic:Conn_01x02
- added Q5: 2N7002, Package_TO_SOT_SMD:SOT-23, symbol Device:Q_NMOS_DGS
- added Q6: SST4401, Package_TO_SOT_SMD:SOT-23, symbol Device:Q_NPN_BCE
- added Q8: NSS60201LT1G, Package_TO_SOT_SMD:SOT-23, symbol Device:Q_NPN_BCE
- added R1: 8k, Resistor_SMD:R_0402_1005Metric, symbol Device:R
- added R13: 10k, Resistor_SMD:R_0402_1005Metric, symbol Device:R
- added R2: 8, Resistor_SMD:R_0402_1005Metric, symbol Device:R
- C24: value 100uF -> 100nF
- C9: value 0.01uF -> 0.1uF
- R10: value 20 -> 5
- R23: value R_Small -> 5k
Connections:
- net labels added: LED_CONTROL, LED_OUT, SOLENOID_GND, SOLENOID_ON
- wire segments 170 -> 168
Other:
- moved on the sheet: C14, C15, C16, C17, C18, C19, C20, C21, C22, C23, C24, C25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

Commit message: Add files via upload
Parts:
- removed C1: 0.1uF, Capacitor_SMD:C_0402_1005Metric, symbol Device:C
- removed C10, C13: 2.2uF, Capacitor_SMD:C_0402_1005Metric, symbol Device:C_Small
- removed C11, C12, C8: 0.01uF, Capacitor_SMD:C_0402_1005Metric, symbol Device:C_Small
- removed C14, C15: 220nF, Capacitor_SMD:C_0402_1005Metric, symbol Device:C_Small
- removed C16, C17: 200nF, Capacitor_SMD:C_0402_1005Metric, symbol Device:C_Small
- removed C18, C19, C20, C21: 100nF, Capacitor_SMD:C_0402_1005Metric, symbol Device:C_Small
- removed C2, C3: 0.47 uF, Capacitor_SMD:C_0402_1005Metric, symbol Device:C_Small
- removed C22, C23: 1nF, Capacitor_SMD:C_0402_1005Metric, symbol Device:C_Small
- removed C24: 100nF, Capacitor_SMD:C_Elec_6.3x7.7, symbol Device:CP_Small
- removed C25: 1000u, Capacitor_THT:C_Radial_D10.0mm_H16.0mm_P5.00mm, symbol Device:CP_Small
- removed C4, C5: 22uF, Capacitor_SMD:C_0402_1005Metric, symbol Device:C_Small
- removed C6: 22uF, Capacitor_SMD:CP_Elec_4x5.8, symbol Device:C
- removed C9: 0.1uF, Capacitor_SMD:C_0402_1005Metric, symbol Device:C_Small
- removed D1: 10V, Diode_SMD:D_SOD-123, symbol Diode:BZT52Bxx
- removed D2: 39V, Diode_SMD:D_SOD-123, symbol Diode:BZT52Bxx
- removed D3, D4: 12V, Diode_SMD:D_SMA, symbol Device:D_Schottky
- removed D5, D6: 5V, Diode_SMD:D_SMA, symbol Device:D_Schottky
- removed D7: MMSD4148, Diode_SMD:D_SOD-123, symbol Device:D
- removed D8: CMPD914E, Package_TO_SOT_SMD:SOT-23, symbol Device:D
- removed F1: TR/3216FF25-R, Fuse:Fuse_1206_3216Metric, symbol Device:Fuse
- removed J1: Conn_01x08, Connector_Molex:Molex_KK-254_AE-6410-08A_1x08_P2.54mm_Vertical, symbol Connector_Generic:Conn_01x08
- removed J10, J3: Conn_01x04, Connector_Molex:Molex_KK-254_AE-6410-04A_1x04_P2.54mm_Vertical, symbol Connector_Generic:Conn_01x04
- removed J2: Laser 1, MJ1-2533-SMT:CUI_MJ1-2533-SMT, symbol Connector_Generic:Conn_01x02
- removed J4, J5, J7: Conn_01x02, Connector_Molex:Molex_KK-254_AE-6410-02A_1x02_P2.54mm_Vertical, symbol Connector_Generic:Conn_01x02
- removed J6: 76825-0006, connector:Molex-76825-0006-0, symbol eec:76825-0006
- removed K1: J115F11AH12VDCS61.5U, Relay_THT:Relay_StandexMeder_UMS, symbol Relay:UMS05-1A80-75L
- removed L1, L2: 4.3 uH, Inductor_SMD:L_Bourns-SRN6028, symbol Device:L
- removed Q1, Q2: BTN8982TA, Package_TO_SOT_SMD:TO-263-7_TabPin8, symbol Power_Management:BTN8982TA
- removed Q3: SUD50P04-08, Package_TO_SOT_SMD:TO-252-2, symbol Transistor_FET:SUD50P04-08
- removed Q4: TIP35CW, Package_TO_SOT_THT:TO-247-3_Vertical, symbol Device:Q_NPN_BCE
- removed Q5: 2N7002, Package_TO_SOT_SMD:SOT-23, symbol Device:Q_NMOS_DGS
- removed Q6: SST4401, Package_TO_SOT_SMD:SOT-23, symbol Device:Q_NPN_BCE
- removed Q8: NSS60201LT1G, Package_TO_SOT_SMD:SOT-23, symbol Device:Q_NPN_BCE
- removed R1: 8k, Resistor_SMD:R_0402_1005Metric, symbol Device:R
- removed R11, R30: 365, Resistor_SMD:R_0402_1005Metric, symbol Device:R_Small
- removed R12, R18: 1.91k, Resistor_SMD:R_0402_1005Metric, symbol Device:R_Small
- removed R13: 10k, Resistor_SMD:R_0402_1005Metric, symbol Device:R
- removed R19, R8: 510, Resistor_SMD:R_0402_1005Metric, symbol Device:R_Small
- removed R2: 8, Resistor_SMD:R_0402_1005Metric, symbol Device:R
- removed R20, R21: 1k, Resistor_SMD:R_0402_1005Metric, symbol Device:R_Small
- removed R22: 10k, Resistor_SMD:R_0402_1005Metric, symbol Device:R_Small
- removed R23: 5k, Resistor_SMD:R_0402_1005Metric, symbol Device:R_Small
- removed R25, R26, R3, R4: 51k, Resistor_SMD:R_0402_1005Metric, symbol Device:R_Small
- removed R27, R5: 47k, Resistor_SMD:R_0402_1005Metric, symbol Device:R_Small
- removed R28, R6: 200k, Resistor_SMD:R_0402_1005Metric, symbol Device:R_Small
- removed R29, R7: 82k, Resistor_SMD:R_0402_1005Metric, symbol Device:R_Small
- removed R31, R32, R33, R34: 6.6k, Resistor_SMD:R_0402_1005Metric, symbol Device:R_Small
- removed R9: 20k, Resistor_SMD:R_0402_1005Metric, symbol Device:R_Small
- removed U1, U9: DRV8834, Package_SO:HTSSOP-24-1EP_4.4x7.8mm_P0.65mm_EP3.2x5mm, symbol Driver_Motor:DRV8834
- removed U2: LT3501, Package_SO:HTSSOP-20-1EP_4.4x6.5mm_P0.65mm_EP3.4x6.5mm_Mask2.75x3.43mm_ThermalVias, symbol Regulator_Switching:LT3501
- removed XA1: Arduino_Due_Shield, Arduino:Arduino_Due_Shield, symbol arduino:Arduino_Due_Shield
- added C?: 10 nF, symbol Device:C_Small
- added C?: 4.7 uF, symbol Device:C_Small
- added C?: 0.1 uF, symbol Device:C_Small
- added C?: 1 uF, symbol Device:C_Small
- added C?: 47 uF, symbol Device:C_Small
- added C?: 10 pF, symbol Device:C_Small
- added J1: Stepper 1 In, symbol Connector_Generic:Conn_01x03
- added J?: Conn_01x01, symbol Connector_Generic:Conn_01x01
- added J?: Stepper 2 In, symbol Connector_Generic:Conn_01x03
- added J?: Laser In, symbol Connector_Generic:Conn_01x02
- added J?: Laser Out, symbol Connector_Generic:Conn_01x02
- added J?: Motor 1 Out, symbol Connector_Generic:Conn_01x02
- added J?: Motor 2 Out, symbol Connector_Generic:Conn_01x02
- added J?: Motor 1 In, symbol Connector_Generic:Conn_01x03
- added J?: Motor 2 Out, symbol Connector_Generic:Conn_01x03
- added J?: Stepper 2 Out, symbol Connector_Generic:Conn_01x04
- added J?: Stepper 1 Out, symbol Connector_Generic:Conn_01x04
- added J?: From Arduino, symbol Connector_Generic:Conn_01x04
- added J?: Conn_01x06, symbol Connector_Generic:Conn_01x06
- added L?: 4.7 uH, symbol Device:L_Small
- added Q? (x6): Q_NPN_BCE, symbol Device:Q_NPN_BCE
- added R? (x4): 1k, symbol Device:R
- added R? (x4): 10k, symbol Device:R
- added R?: 20, symbol Device:R
- added R?: 60.4K, symbol Device:R_Small
- added R?: 1M, symbol Device:R_Small
- added R?: 243K, symbol Device:R_Small
- added U? (x3): L293D, Package_DIP:DIP-16_W7.62mm, symbol Driver_Motor:L293D
- added U?: LT8610, Package_SO:LTC_MSOP-16-1EP_3x4mm_P0.5mm_EP2.15x3.26mm, symbol Regulator_Switching:LT8610
- C?: renamed from C7; footprint Capacitor_SMD:CP_Elec_3x5.3 -> (none)
- Q?: renamed from Q7; footprint Package_TO_SOT_SMD:SOT-23 -> (none)
- R?: renamed from R14; value 4 -> 4.16; footprint Resistor_SMD:R_0402_1005Metric -> (none)
- R?: renamed from R10; value 5 -> 20; footprint Resistor_SMD:R_0402_1005Metric -> (none)
- R?: renamed from R15; footprint Resistor_SMD:R_0402_1005Metric -> (none)
Connections:
- net labels added: +24V, 24V, LASER2_CONTROL, LASER2_OUT, MOTOR1_CONTROL1, MOTOR1_CONTROL2, MOTOR1_ENABLE, MOTOR1_OUT1, MOTOR1_OUT2, MOTOR2_CONTROL1, MOTOR2_CONTROL2, MOTOR2_ENABLE, MOTOR2_OUT1, MOTOR2_OUT2, STEPPER1_2A, STEPPER1_3A, STEPPER1_CONTROL1, STEPPER1_CONTROL2, STEPPER1_ENABLE, STEPPER2_2A, STEPPER2_3A, STEPPER2_CONTROL1, STEPPER2_CONTROL2, STEPPER2_ENABLE, SUCCESS_OUT
- net labels removed: 12V, 12V_in, 5V(Steppers), AD_1, AD_2, BST1, BST2, FB1, FB2, IO_1_IN_2, IO_2_IN_1, IO_3_INH_2, IO_4_INH_1, LED_CONTROL, LED_OUT, MOTOR_OUT1, MOTOR_OUT2, OTHER_LINE_OK, POWER_ON, REG_SHUTDOWN, SOFT_START, SOLENOID_GND, SOLENOID_ON, STEPPER1_DIRECTION, STEPPER1_STEP, STEPPER1_notENABLE, STEPPER2_DIRECTION, STEPPER2_STEP, STEPPER2_notENABLE, STEPPER_LINE_OK, VINT_OUT, VINT_OUT2, VREF(1.45V), VREF2(1.45V), Vmotor, notFAULT1, notFAULT2
- wire segments 168 -> 55
Other:
- moved on the sheet: C?, R?

Commit message: Add files via upload
Parts:
- removed C?: 10 nF, symbol Device:C_Small
- removed C?: 4.7 uF, symbol Device:C_Small
- removed C?: 0.1 uF, symbol Device:C_Small
- removed C?: 1 uF, symbol Device:C_Small
- removed C?: 47 uF, symbol Device:C_Small
- removed C?: 10 pF, symbol Device:C_Small
- removed J1: Stepper 1 In, symbol Connector_Generic:Conn_01x03
- removed J?: Conn_01x01, symbol Connector_Generic:Conn_01x01
- removed J?: Stepper 2 In, symbol Connector_Generic:Conn_01x03
- removed J?: Laser In, symbol Connector_Generic:Conn_01x02
- removed J?: Laser Out, symbol Connector_Generic:Conn_01x02
- removed J?: Motor 1 Out, symbol Connector_Generic:Conn_01x02
- removed J?: Motor 2 Out, symbol Connector_Generic:Conn_01x02
- removed J?: Motor 1 In, symbol Connector_Generic:Conn_01x03
- removed J?: Motor 2 Out, symbol Connector_Generic:Conn_01x03
- removed J?: Stepper 2 Out, symbol Connector_Generic:Conn_01x04
- removed J?: Stepper 1 Out, symbol Connector_Generic:Conn_01x04
- removed J?: From Arduino, symbol Connector_Generic:Conn_01x04
- removed J?: Conn_01x06, symbol Connector_Generic:Conn_01x06
- removed L?: 4.7 uH, symbol Device:L_Small
- removed Q? (x6): Q_NPN_BCE, symbol Device:Q_NPN_BCE
- removed R? (x4): 1k, symbol Device:R
- removed R? (x4): 10k, symbol Device:R
- removed R?: 20, symbol Device:R
- removed R?: 60.4K, symbol Device:R_Small
- removed R?: 1M, symbol Device:R_Small
- removed R?: 243K, symbol Device:R_Small
- removed U? (x3): L293D, Package_DIP:DIP-16_W7.62mm, symbol Driver_Motor:L293D
- removed U?: LT8610, Package_SO:LTC_MSOP-16-1EP_3x4mm_P0.5mm_EP2.15x3.26mm, symbol Regulator_Switching:LT8610
- added C1: 0.1uF, Capacitor_SMD:C_0402_1005Metric, symbol Device:C
- added C10, C13: 2.2uF, Capacitor_SMD:C_0402_1005Metric, symbol Device:C_Small
- added C11, C12, C8: 0.01uF, Capacitor_SMD:C_0402_1005Metric, symbol Device:C_Small
- added C14, C15: 220nF, Capacitor_SMD:C_0402_1005Metric, symbol Device:C_Small
- added C16, C17: 200nF, Capacitor_SMD:C_0402_1005Metric, symbol Device:C_Small
- added C18, C19, C20, C21: 100nF, Capacitor_SMD:C_0402_1005Metric, symbol Device:C_Small
- added C2, C3: 0.47 uF, Capacitor_SMD:C_0402_1005Metric, symbol Device:C_Small
- added C22, C23: 1nF, Capacitor_SMD:C_0402_1005Metric, symbol Device:C_Small
- added C24: 100nF, Capacitor_SMD:C_Elec_6.3x7.7, symbol Device:CP_Small
- added C25: 1000u, Capacitor_THT:C_Radial_D10.0mm_H16.0mm_P5.00mm, symbol Device:CP_Small
- added C4, C5: 22uF, Capacitor_SMD:C_0402_1005Metric, symbol Device:C_Small
- added C6: 22uF, Capacitor_SMD:CP_Elec_4x5.8, symbol Device:C
- added C9: 0.1uF, Capacitor_SMD:C_0402_1005Metric, symbol Device:C_Small
- added D1: 10V, Diode_SMD:D_SOD-123, symbol Diode:BZT52Bxx
- added D2: 39V, Diode_SMD:D_SOD-123, symbol Diode:BZT52Bxx
- added D3, D4: 12V, Diode_SMD:D_SMA, symbol Device:D_Schottky
- added D5, D6: 5V, Diode_SMD:D_SMA, symbol Device:D_Schottky
- added D7: MMSD4148, Diode_SMD:D_SOD-123, symbol Device:D
- added D8: CMPD914E, Package_TO_SOT_SMD:SOT-23, symbol Device:D
- added F1: TR/3216FF25-R, Fuse:Fuse_1206_3216Metric, symbol Device:Fuse
- added J1: Conn_01x08, Connector_Molex:Molex_KK-254_AE-6410-08A_1x08_P2.54mm_Vertical, symbol Connector_Generic:Conn_01x08
- added J10, J3: Conn_01x04, Connector_Molex:Molex_KK-254_AE-6410-04A_1x04_P2.54mm_Vertical, symbol Connector_Generic:Conn_01x04
- added J2: Laser 1, MJ1-2533-SMT:CUI_MJ1-2533-SMT, symbol Connector_Generic:Conn_01x02
- added J4, J5, J7: Conn_01x02, Connector_Molex:Molex_KK-254_AE-6410-02A_1x02_P2.54mm_Vertical, symbol Connector_Generic:Conn_01x02
- added J6: 76825-0006, connector:Molex-76825-0006-0, symbol eec:76825-0006
- added K1: J115F11AH12VDCS61.5U, Relay_THT:Relay_StandexMeder_UMS, symbol Relay:UMS05-1A80-75L
- added L1, L2: 4.3 uH, Inductor_SMD:L_Bourns-SRN6028, symbol Device:L
- added Q1, Q2: BTN8982TA, Package_TO_SOT_SMD:TO-263-7_TabPin8, symbol Power_Management:BTN8982TA
- added Q3: SUD50P04-08, Package_TO_SOT_SMD:TO-252-2, symbol Transistor_FET:SUD50P04-08
- added Q4: TIP35CW, Package_TO_SOT_THT:TO-247-3_Vertical, symbol Device:Q_NPN_BCE
- added Q5: 2N7002, Package_TO_SOT_SMD:SOT-23, symbol Device:Q_NMOS_DGS
- added Q6: SST4401, Package_TO_SOT_SMD:SOT-23, symbol Device:Q_NPN_BCE
- added Q8: NSS60201LT1G, Package_TO_SOT_SMD:SOT-23, symbol Device:Q_NPN_BCE
- added R1: 8k, Resistor_SMD:R_0402_1005Metric, symbol Device:R
- added R11, R30: 365, Resistor_SMD:R_0402_1005Metric, symbol Device:R_Small
- added R12, R18: 1.91k, Resistor_SMD:R_0402_1005Metric, symbol Device:R_Small
- added R13: 10k, Resistor_SMD:R_0402_1005Metric, symbol Device:R
- added R19, R8: 510, Resistor_SMD:R_0402_1005Metric, symbol Device:R_Small
- added R2: 8, Resistor_SMD:R_0402_1005Metric, symbol Device:R
- added R20, R21: 1k, Resistor_SMD:R_0402_1005Metric, symbol Device:R_Small
- added R22: 10k, Resistor_SMD:R_0402_1005Metric, symbol Device:R_Small
- added R23: 5k, Resistor_SMD:R_0402_1005Metric, symbol Device:R_Small
- added R25, R26, R3, R4: 51k, Resistor_SMD:R_0402_1005Metric, symbol Device:R_Small
- added R27, R5: 47k, Resistor_SMD:R_0402_1005Metric, symbol Device:R_Small
- added R28, R6: 200k, Resistor_SMD:R_0402_1005Metric, symbol Device:R_Small
- added R29, R7: 82k, Resistor_SMD:R_0402_1005Metric, symbol Device:R_Small
- added R31, R32, R33, R34: 6.6k, Resistor_SMD:R_0402_1005Metric, symbol Device:R_Small
- added R9: 20k, Resistor_SMD:R_0402_1005Metric, symbol Device:R_Small
- added U1, U9: DRV8834, Package_SO:HTSSOP-24-1EP_4.4x7.8mm_P0.65mm_EP3.2x5mm, symbol Driver_Motor:DRV8834
- added U2: LT3501, Package_SO:HTSSOP-20-1EP_4.4x6.5mm_P0.65mm_EP3.4x6.5mm_Mask2.75x3.43mm_ThermalVias, symbol Regulator_Switching:LT3501
- added XA1: Arduino_Due_Shield, Arduino:Arduino_Due_Shield, symbol arduino:Arduino_Due_Shield
- C7: renamed from C?; footprint (none) -> Capacitor_SMD:CP_Elec_3x5.3
- Q7: renamed from Q?; footprint (none) -> Package_TO_SOT_SMD:SOT-23
- R10: renamed from R?; value 20 -> 5; footprint (none) -> Resistor_SMD:R_0402_1005Metric
- R14: renamed from R?; value 4.16 -> 4; footprint (none) -> Resistor_SMD:R_0402_1005Metric
- R15: renamed from R?; footprint (none) -> Resistor_SMD:R_0402_1005Metric
Connections:
- net labels added: 12V, 12V_in, 5V(Steppers), AD_1, AD_2, BST1, BST2, FB1, FB2, IO_1_IN_2, IO_2_IN_1, IO_3_INH_2, IO_4_INH_1, LED_CONTROL, LED_OUT, MOTOR_OUT1, MOTOR_OUT2, OTHER_LINE_OK, POWER_ON, REG_SHUTDOWN, SOFT_START, SOLENOID_GND, SOLENOID_ON, STEPPER1_DIRECTION, STEPPER1_STEP, STEPPER1_notENABLE, STEPPER2_DIRECTION, STEPPER2_STEP, STEPPER2_notENABLE, STEPPER_LINE_OK, VINT_OUT, VINT_OUT2, VREF(1.45V), VREF2(1.45V), Vmotor, notFAULT1, notFAULT2
- net labels removed: +24V, 24V, LASER2_CONTROL, LASER2_OUT, MOTOR1_CONTROL1, MOTOR1_CONTROL2, MOTOR1_ENABLE, MOTOR1_OUT1, MOTOR1_OUT2, MOTOR2_CONTROL1, MOTOR2_CONTROL2, MOTOR2_ENABLE, MOTOR2_OUT1, MOTOR2_OUT2, STEPPER1_2A, STEPPER1_3A, STEPPER1_CONTROL1, STEPPER1_CONTROL2, STEPPER1_ENABLE, STEPPER2_2A, STEPPER2_3A, STEPPER2_CONTROL1, STEPPER2_CONTROL2, STEPPER2_ENABLE, SUCCESS_OUT
- wire segments 55 -> 168
Other:
- moved on the sheet: C7, R10, R14, R15
