File: Projects/ScienceBoard-2/ScienceBoard-1.sch (KiCad schematic (older format))
At the start: 88 parts, among them J1 Conn_01x08, J10 Conn_01x04, J2 Laser 1, J3 Conn_01x04, J4 Conn_01x02, J5 Conn_01x02, J6 76825-0006, J7 Conn_01x02, K1 J115F11AH12VDCS61.5U, Q1 BTN8982TA, Q2 BTN8982TA, Q3 SUD50P04-08, Q4 TIP35CW, Q5 2N7002, Q6 SST4401, Q7 Q_PNP_BCE, Q8 NSS60201LT1G, U1 DRV8834, U2 LT3501, U9 DRV8834

Commit message: Add files via upload
Parts:
- removed Q5: 2N7002, Package_TO_SOT_SMD:SOT-23, symbol Device:Q_NMOS_DGS
- removed R14: 4, Resistor_SMD:R_0402_1005Metric, symbol Device:R_Small
- added C26: 4.7 uF, Capacitor_SMD:C_0402_1005Metric, symbol Device:CP
- added C27: 47 uF, Capacitor_SMD:C_0402_1005Metric, symbol Device:CP
- added Q5: FMMT634Q, Package_TO_SOT_SMD:SOT-23, symbol Device:Q_NPN_BCE
- added R14: 1k, Resistor_SMD:R_0402_1005Metric, symbol Device:R
- added R16: 3k, Resistor_SMD:R_0402_1005Metric, symbol Device:R
- added R17: 20k, Resistor_SMD:R_0402_1005Metric, symbol Device:R
- added R24: 20, Resistor_SMD:R_0402_1005Metric, symbol Device:R
- added U3: NCP57302, Package_TO_SOT_SMD:TO-252-5_TabPin3, symbol Regulator_Linear:NCP57302
- C12: value 0.01uF -> 0.1uF
Connections:
- net 5V: now also C7.1, C26.1, U3.1 (EN), U3.2 (VIN); no longer C7.2
- net GND: now also C7.2, C26.2, C27.2, Q5.3 (E), R16.2, U3.3 (GND); no longer C7.1
- net ICG: now also XA1.D9; no longer XA1.D14 (D14_TX3)
- net OutputSignal_out: now also XA1.A3; no longer XA1.D15 (D15_RX3), XA1.D34
- net SH: now also XA1.D10 (D10_CS0); no longer XA1.D17 (D17_RX2)
- net SOLENOID_GND: now also R24.1
- net SOLENOID_ON: now also R17.2
- net VPELT: now also C27.1, R14.1, U3.4 (VOUT)
- net phiM(CCD_Clock): now also XA1.D2; no longer XA1.D16 (D16_TX2)
- new net: R14.2, R16.1, U3.5 (ADJ)
- new net: Q5.1 (B), R17.1
- new net: Q5.2 (C), R24.2
Changed lines of the file:
@@
 Text Label 7700 5200 0    50   ~ 0
 OutputSignal_in
-Text Label 11850 3550 2    50   ~ 0
-OutputSignal_out
-Text Label 14450 5450 0    50   ~ 0
+Text Label 11850 5950 2    50   ~ 0
 phiM(CCD_Clock)
-Text Label 14450 5550 0    50   ~ 0
+Text Label 11850 5150 2    50   ~ 0
 SH
-Text Label 14450 5250 0    50   ~ 0
+Text Label 11850 5250 2    50   ~ 0
 ICG
 $Comp
@@
 F 3 "~" H 7050 6200 50  0001 C CNN
 	1    7050 6200
-	1    0    0    -1
+	-1   0    0    1
 $EndComp
 Text Label 6250 6350 2    50   ~ 0
@@
 Wire Notes Line
 	8450 4850 8450 7300
-$Comp
-L Device:R_Small R14
-U 1 1 5FBBBE3B
-P 6350 5950
-F 0 "R14" V 6154 5950 50  0000 C CNN
-F 1 "4" V 6245 5950 50  0000 C CNN
-F 2 "Resistor_SMD:R_0402_1005Metric" H 6350 5950 50  0001 C CNN
-F 3 "~" H 6350 5950 50  0001 C CNN
-	1    6350 5950
-	0    1    1    0
-$EndComp
-Text Label 6250 5950 2    50   ~ 0
-5V
-Text Label 6450 5950 0    50   ~ 0
-VPELT
 Wire Notes Line
 	5850 4850 8450 4850
@@
 P 3900 5450
 F 0 "C12" H 3992 5496 50  0000 L CNN
-F 1 "0.01uF" H 3992 5405 50  0000 L CNN
+F 1 "0.1uF" H 3992 5405 50  0000 L CNN
 F 2 "Capacitor_SMD:C_0402_1005Metric" H 3900 5450 50  0001 C CNN
 F 3 "~" H 3900 5450 50  0001 C CNN
@@
 Text Label 11850 2550 2    50   ~ 0
 STEPPER1_notENABLE
-Text Label 14450 5350 0    50   ~ 0
+Text Label 14450 3950 0    50   ~ 0
 OutputSignal_out
 $Comp
@@
 	7900 1400 7700 1400
 $Comp
-L Device:Q_NMOS_DGS Q5
-U 1 1 608F6C24
-P 9850 3850
-F 0 "Q5" H 10056 3804 50  0000 L CNN
-F 1 "2N7002" H 10056 3895 50  0000 L CNN
-F 2 "Package_TO_SOT_SMD:SOT-23" H 10050 3950 50  0001 C CNN
-F 3 "~" H 9850 3850 50  0001 C CNN
-	1    9850 3850
-	-1   0    0    1
-$EndComp
-Text Label 10050 3850 0    50   ~ 0
-SOLENOID_ON
-$Comp
 L Connector_Generic:Conn_01x02 J5
 U 1 1 60901E57
@@
 Text Label 10250 4600 0    50   ~ 0
 12V
-$Comp
-L power:GND #PWR0158
-U 1 1 60908998
-P 9750 4050
-F 0 "#PWR0158" H 9750 3800 50  0001 C CNN
-F 1 "GND" H 9755 3877 50  0000 C CNN
-F 2 "" H 9750 4050 50  0001 C CNN
-F 3 "" H 9750 4050 50  0001 C CNN
-	1    9750 4050
-	1    0    0    -1
-$EndComp
-Text Label 9750 3650 0    50   ~ 0
-SOLENOID_GND
 $Comp
 L power:GND #PWR0101
@@
 Text Label 14450 4150 0    50   ~ 0
 AD_2
+$Comp
+L Regulator_Linear:NCP57302 U3
+U 1 1 609AABC8
+P 6950 8200
+F 0 "U3" H 6950 8665 50  0000 C CNN
+F 1 "NCP57302" H 6950 8574 50  0000 C CNN
+F 2 "Package_TO_SOT_SMD:TO-252-5_TabPin3" H 6950 7500 50  0001 C CNN
+F 3 "" H 6950 7500 50  0001 C CNN
+	1    6950 8200
+	1    0    0    -1
+$EndComp
+$Comp
+L Device:CP C26
+U 1 1 609AD41E
+P 6000 8150
+F 0 "C26" H 6118 8196 50  0000 L CNN
+F 1 "4.7 uF" H 6118 8105 50  0000 L CNN
+F 2 "Capacitor_SMD:C_0402_1005Metric" H 6038 8000 50  0001 C CNN
+F 3 "~" H 6000 8150 50  0001 C CNN
+	1    6000 8150
+	1    0    0    -1
+$EndComp
+$Comp
+L Device:R R14
+U 1 1 609C36CC
+P 7600 8150
+F 0 "R14" H 7670 8196 50  0000 L CNN
+F 1 "1k" H 7670 8105 50  0000 L CNN
+F 2 "Resistor_SMD:R_0402_1005Metric" V 7530 8150 50  0001 C CNN
+F 3 "~" H 7600 8150 50  0001 C CNN
+	1    7600 8150
+	1    0    0    -1
+$EndComp
+$Comp
+L Device:R R16
+U 1 1 609C4750
+P 7600 8650
+F 0 "R16" H 7670 8696 50  0000 L CNN
+F 1 "3k" H 7670 8605 50  0000 L CNN
+F 2 "Resistor_SMD:R_0402_1005Metric" V 7530 8650 50  0001 C CNN
+F 3 "~" H 7600 8650 50  0001 C CNN
+	1    7600 8650
+	1    0    0    -1
+$EndComp
+Wire Wire Line
+	7600 8500 7600 8400
+Wire Wire Line
+	7350 8400 7600 8400
+Connection ~ 7600 8400
+Wire Wire Line
+	7600 8400 7600 8300
+$Comp
+L Device:CP C27
+U 1 1 609D5663
+P 8100 8150
+F 0 "C27" H 8218 8196 50  0000 L CNN
+F 1 "47 uF" H 8218 8105 50  0000 L CNN
+F 2 "Capacitor_SMD:C_0402_1005Metric" H 8138 8000 50  0001 C CNN
+F 3 "~" H 8100 8150 50  0001 C CNN
+	1    8100 8150
+	1    0    0    -1
+$EndComp
+Wire Wire Line
+	6000 8000 6400 8000
+Wire Wire Line
+	6400 8000 6400 8400
+Wire Wire Line
+	6400 8400 6550 8400
+Connection ~ 6400 8000
+Wire Wire Line
+	6400 8000 6550 8000
+Wire Wire Line
+	7350 8000 7600 8000
+Connection ~ 7600 8000
+Wire Wire Line
+	7600 8000 8100 8000
+$Comp
+L power:GND #PWR0160
+U 1 1 60A07C53
+P 6950 8600
+F 0 "#PWR0160" H 6950 8350 50  0001 C CNN
+F 1 "GND" H 6955 8427 50  0000 C CNN
+F 2 "" H 6950 8600 50  0001 C CNN
+F 3 "" H 6950 8600 50  0001 C CNN
+	1    6950 8600
+	1    0    0    -1
+$EndComp
+$Comp
+L power:GND #PWR0161
+U 1 1 60A08D75
+P 8100 8300
+F 0 "#PWR0161" H 8100 8050 50  0001 C CNN
+F 1 "GND" H 8105 8127 50  0000 C CNN
+F 2 "" H 8100 8300 50  0001 C CNN
+F 3 "" H 8100 8300 50  0001 C CNN
+	1    8100 8300
+	1    0    0    -1
+$EndComp
+$Comp
+L power:GND #PWR0162
+U 1 1 60A09A33
+P 6000 8300
+F 0 "#PWR0162" H 6000 8050 50  0001 C CNN
+F 1 "GND" H 6005 8127 50  0000 C CNN
+F 2 "" H 6000 8300 50  0001 C CNN
+F 3 "" H 6000 8300 50  0001 C CNN
+	1    6000 8300
+	1    0    0    -1
+$EndComp
+$Comp
+L power:GND #PWR0163
+U 1 1 60A0AAC6
+P 7600 8800
+F 0 "#PWR0163" H 7600 8550 50  0001 C CNN
+F 1 "GND" H 7605 8627 50  0000 C CNN
+F 2 "" H 7600 8800 50  0001 C CNN
+F 3 "" H 7600 8800 50  0001 C CNN
+	1    7600 8800
+	1    0    0    -1
+$EndComp
+Text Label 5800 8000 2    50   ~ 0
+5V
+Wire Wire Line
+	6000 8000 5800 8000
+Connection ~ 6000 8000
+Text Label 8250 8000 0    50   ~ 0
+VPELT
+Wire Wire Line
+	8250 8000 8100 8000
+Connection ~ 8100 8000
+$Comp
+L Device:Q_NPN_BCE Q5
+U 1 1 60A378CC
+P 10300 3950
+F 0 "Q5" H 10490 3996 50  0000 L CNN
+F 1 "FMMT634Q" H 10490 3905 50  0000 L CNN
+F 2 "Package_TO_SOT_SMD:SOT-23" H 10500 4050 50  0001 C CNN
+F 3 "~" H 10300 3950 50  0001 C CNN
+	1    10300 3950
+	1    0    0    -1
+$EndComp
+$Comp
+L power:GND #PWR0158
+U 1 1 60A44E6B
+P 10400 4150
+F 0 "#PWR0158" H 10400 3900 50  0001 C CNN
+F 1 "GND" H 10405 3977 50  0000 C CNN
+F 2 "" H 10400 4150 50  0001 C CNN
+F 3 "" H 10400 4150 50  0001 C CNN
+	1    10400 4150
+	1    0    0    -1
+$EndComp
+Text Label 9800 3950 2    50   ~ 0
+SOLENOID_ON
+Text Label 10400 3450 0    50   ~ 0
+SOLENOID_GND
+$Comp
+L Device:R R24
+U 1 1 60A469F3
+P 10400 3600
+F 0 "R24" H 10470 3646 50  0000 L CNN
+F 1 "20" H 10470 3555 50  0000 L CNN
+F 2 "Resistor_SMD:R_0402_1005Metric" V 10330 3600 50  0001 C CNN
+F 3 "~" H 10400 3600 50  0001 C CNN
+	1    10400 3600
+	1    0    0    -1
+$EndComp
+$Comp
+L Device:R R17
+U 1 1 60A43884
+P 9950 3950
+F 0 "R17" V 9743 3950 50  0000 C CNN
+F 1 "20k" V 9834 3950 50  0000 C CNN
+F 2 "Resistor_SMD:R_0402_1005Metric" V 9880 3950 50  0001 C CNN
+F 3 "~" H 9950 3950 50  0001 C CNN
+	1    9950 3950
+	0    1    1    0
+$EndComp
 $EndSCHEMATC

Commit message: Add files via upload
Parts:
- removed C1: 0.1uF, Capacitor_SMD:C_0402_1005Metric, symbol Device:C
- removed C2, C3: 0.47 uF, Capacitor_SMD:C_0402_1005Metric, symbol Device:C_Small
- removed C4, C5: 22uF, Capacitor_SMD:C_0402_1005Metric, symbol Device:C_Small
- removed C6: 22uF, Capacitor_SMD:CP_Elec_4x5.8, symbol Device:C
- removed D3, D4: 12V, Diode_SMD:D_SMA, symbol Device:D_Schottky
- removed D5, D6: 5V, Diode_SMD:D_SMA, symbol Device:D_Schottky
- removed L1, L2: 4.3 uH, Inductor_SMD:L_Bourns-SRN6028, symbol Device:L
- removed R11, R30: 365, Resistor_SMD:R_0402_1005Metric, symbol Device:R_Small
- removed R12, R18: 1.91k, Resistor_SMD:R_0402_1005Metric, symbol Device:R_Small
- removed R9: 20k, Resistor_SMD:R_0402_1005Metric, symbol Device:R_Small
- removed U2: LT3501, Package_SO:HTSSOP-20-1EP_4.4x6.5mm_P0.65mm_EP3.4x6.5mm_Mask2.75x3.43mm_ThermalVias, symbol Regulator_Switching:LT3501
- added J8: Conn_01x06, Connector_Molex:Molex_KK-254_AE-6410-06A_1x06_P2.54mm_Vertical, symbol Connector_Generic:Conn_01x06
Connections:
- net 5V(Steppers) is gone; now on net 5V: C11.1, C12.1, C8.1, C9.1, R27.2, R28.1, R5.2, R6.1, U1.17 (VCP), U1.18 (VM), U1.19 (VM), U9.17 (VCP), U9.18 (VM), U9.19 (VM)
- net 12V: now also J8.1 (Pin_1), J8.2 (Pin_2)
- net 5V: now also J8.5 (Pin_5), J8.6 (Pin_6)
- net GND: now also J8.3 (Pin_3), J8.4 (Pin_4)
- net OTHER_LINE_OK: no longer names the net of XA1.D53
- net REG_SHUTDOWN: no longer names the net of XA1.D7
- net STEPPER_LINE_OK: no longer names the net of XA1.D52 (D52_CS2)

Commit message: Add files via upload
Parts:
- added J11, J9: Conn_01x02, Connector_Molex:Molex_KK-254_AE-6410-02A_1x02_P2.54mm_Vertical, symbol Connector_Generic:Conn_01x02
Connections:
- net GND: now also J11.2 (Pin_2), J9.2 (Pin_2)
- net ICG: now also XA1.D21 (D21_SCL); no longer XA1.D9
- net SH: now also XA1.D20 (D20_SDA); no longer XA1.D10 (D10_CS0)
- net phiM(CCD_Clock): now also XA1.D16 (D16_TX2); no longer XA1.D2
- net LIMIT_SWITCH_1: now reaches XA1.D34
- net LIMIT_SWITCH_1: now also J9.1 (Pin_1)
- net LIMIT_SWITCH_2: now reaches XA1.D52 (D52_CS2)
- net LIMIT_SWITCH_2: now also J11.1 (Pin_1)
Changed lines of the file:
@@
 Text Label 7700 5200 0    50   ~ 0
 OutputSignal_in
-Text Label 11850 5950 2    50   ~ 0
+Text Label 14450 5450 0    50   ~ 0
 phiM(CCD_Clock)
-Text Label 11850 5150 2    50   ~ 0
+Text Label 14450 5150 0    50   ~ 0
 SH
-Text Label 11850 5250 2    50   ~ 0
+Text Label 14450 5050 0    50   ~ 0
 ICG
 $Comp
@@
 Text Label 3300 9300 2    50   ~ 0
 5V
+$Comp
+L Connector_Generic:Conn_01x02 J9
+U 1 1 609ACEEE
+P 1500 8000
+F 0 "J9" H 1580 7992 50  0000 L CNN
+F 1 "Conn_01x02" H 1580 7901 50  0000 L CNN
+F 2 "Connector_Molex:Molex_KK-254_AE-6410-02A_1x02_P2.54mm_Vertical" H 1500 8000 50  0001 C CNN
+F 3 "~" H 1500 8000 50  0001 C CNN
+	1    1500 8000
+	1    0    0    -1
+$EndComp
+$Comp
+L Connector_Generic:Conn_01x02 J11
+U 1 1 609ADE84
+P 1500 8450
+F 0 "J11" H 1580 8442 50  0000 L CNN
+F 1 "Conn_01x02" H 1580 8351 50  0000 L CNN
+F 2 "Connector_Molex:Molex_KK-254_AE-6410-02A_1x02_P2.54mm_Vertical" H 1500 8450 50  0001 C CNN
+F 3 "~" H 1500 8450 50  0001 C CNN
+	1    1500 8450
+	1    0    0    -1
+$EndComp
+$Comp
+L power:GND #PWR0112
+U 1 1 609B515C
+P 1300 8550
+F 0 "#PWR0112" H 1300 8300 50  0001 C CNN
+F 1 "GND" H 1305 8377 50  0000 C CNN
+F 2 "" H 1300 8550 50  0001 C CNN
+F 3 "" H 1300 8550 50  0001 C CNN
+	1    1300 8550
+	1    0    0    -1
+$EndComp
+Text Label 1300 8000 2    50   ~ 0
+LIMIT_SWITCH_1
+Text Label 1300 8450 2    50   ~ 0
+LIMIT_SWITCH_2
+$Comp
+L power:GND #PWR0113
+U 1 1 609B8045
+P 1300 8100
+F 0 "#PWR0113" H 1300 7850 50  0001 C CNN
+F 1 "GND" H 1305 7927 50  0000 C CNN
+F 2 "" H 1300 8100 50  0001 C CNN
+F 3 "" H 1300 8100 50  0001 C CNN
+	1    1300 8100
+	1    0    0    -1
+$EndComp
+Text Label 11850 3550 2    50   ~ 0
+LIMIT_SWITCH_1
+Text Label 11850 1750 2    50   ~ 0
+LIMIT_SWITCH_2
 $EndSCHEMATC

Commit message: Add files via upload
Parts:
- removed C26: 4.7 uF, Capacitor_SMD:C_0402_1005Metric, symbol Device:CP
- removed C27: 47 uF, Capacitor_SMD:C_0402_1005Metric, symbol Device:CP
- removed C7: 10 uF, Capacitor_SMD:CP_Elec_3x5.3, symbol Device:CP
- removed Q7: Q_PNP_BCE, Package_TO_SOT_SMD:SOT-23, symbol Device:Q_PNP_BCE
- removed Q8: NSS60201LT1G, Package_TO_SOT_SMD:SOT-23, symbol Device:Q_NPN_BCE
- removed R14: 1k, Resistor_SMD:R_0402_1005Metric, symbol Device:R
- removed R15: 2.2k, Resistor_SMD:R_0402_1005Metric, symbol Device:R
- removed R16: 3k, Resistor_SMD:R_0402_1005Metric, symbol Device:R
- removed U3: NCP57302, Package_TO_SOT_SMD:TO-252-5_TabPin3, symbol Regulator_Linear:NCP57302
- removed XA1: Arduino_Due_Shield, Arduino:Arduino_Due_Shield, symbol arduino:Arduino_Due_Shield
- added R9: 5.1k, Resistor_SMD:R_0402_1005Metric, symbol Device:R
- added U2, U3: VO14642AT, Package_DIP:VO14642AT, symbol Relay_SolidState:VO14642AT
- added XA2: Arduino_Mega2560_Shield, Arduino:Arduino_Mega2560_Shield, symbol arduino:Arduino_Mega2560_Shield
- Q6: value SST4401 -> FMMT634Q
- R1: value 8k -> 5.1k
Connections:
- net 5V: now also U2.6; no longer J1.4 (Pin_4)
- net AD_1: now also XA2.A0
- net AD_2: now also XA2.A1
- net GND: now also U2.2, U3.2, U3.4; no longer J2.1 (Pin_1)
- net ICG: now also XA2.D21 (D21_SCL)
- net LASER1_CONTROL: now also XA2.D8
- net LASER1_OUT: no longer Q6.2 (C)
- net LED_CONTROL: now also XA2.D4
- net LED_OUT: now also U3.6
- net LIMIT_SWITCH_1: now also XA2.D34
- net LIMIT_SWITCH_2: now also XA2.D52
- net OutputSignal_out: now also J1.4 (Pin_4), XA2.A3
- net POWER_ON: now also XA2.D51
- net SH: now also XA2.D20 (D20_SDA)
- net SOLENOID_ON: now also XA2.D22
- net STEPPER1_DIRECTION: now also XA2.D40
- net STEPPER1_STEP: now also XA2.D42
- net STEPPER1_notENABLE: now also XA2.D44
- net STEPPER2_DIRECTION: now also XA2.D46
- net STEPPER2_STEP: now also XA2.D48
- net STEPPER2_notENABLE: now also XA2.D50
- net VPELT: now also U2.4
- net notFAULT1: now also XA2.D38
- net notFAULT2: now also XA2.D36
- net phiM(CCD_Clock): now also XA2.D2 (D2_INT0)
- net at R32.1: now also XA2.D11
- net at R34.1: now also XA2.D12
- net at R31.2: now also XA2.D13
- net at R33.1: now also XA2.D3 (D3_INT1)
- net at R1.1: now also U3.1
- net OutputSignal_in renamed VCCD
- new net: R9.1, U2.1
- new net LASER1_GND: J2.1 (Pin_1), Q6.2 (C)
- new net PELTIER_ON: R9.2, XA2.D14 (D14_TX3)
Other:
- moved on the sheet: J1, J2, J7, R1, R2
