File: Projects/ScienceBoard-2/ScienceBoard-1.sch (KiCad schematic (older format))
At the start: 73 parts, among them J1 Conn_01x08, J10 Conn_01x04, J11 Conn_01x02, J2 Laser 1, J3 Conn_01x04, J4 Conn_01x02, J5 Conn_01x02, J6 76825-0006, J7 Conn_01x02, J8 Conn_01x06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

Commit message: Add files via upload
Parts:
- removed J6: 76825-0006, connector:Molex-76825-0006-0, symbol eec:76825-0006
- added J6: Conn_01x02, Connector_Molex:Molex_Mega-Fit_76829-0002_2x01_P5.70mm_Vertical, symbol Connector_Generic:Conn_01x02
- J8: footprint Connector_Molex:Molex_KK-254_AE-6410-06A_1x06_P2.54mm_Vertical -> Connector_Molex:Molex_Micro-Fit_3.0_43045-0612_2x03_P3.00mm_Vertical
Connections:
- net 12V: now also J8.4 (Pin_4); no longer J8.2 (Pin_2)
- net 12V_in: now also J6.2 (Pin_2)
- net 5V: now also J8.3 (Pin_3); no longer J8.5 (Pin_5)
- net GND: now also J8.2 (Pin_2), J8.5 (Pin_5), J6.1 (Pin_1); no longer J8.3 (Pin_3), J8.4 (Pin_4)
Changed lines of the file:
@@
-$EndComp
-$Comp
-L eec:76825-0006 J6
-U 1 1 5FE0E70D
-P 6500 1150
-F 0 "J6" H 6258 1515 50  0000 C CNN
-F 1 "76825-0006" H 6258 1424 50  0000 C CNN
-F 2 "connector:Molex-76825-0006-0" H 6500 1650 50  0001 L CNN
-F 3 "https://www.molex.com/pdm_docs/sd/768250006_sd.pdf" H 6500 1750 50  0001 L CNN
-F 4 "Conn" H 6500 1850 50  0001 L CNN "category"
-F 5 "DUAL ROW RA HEADER TIN 6CKT" H 6500 1950 50  0001 L CNN "digikey description"
-F 6 "WM11971-ND" H 6500 2050 50  0001 L CNN "digikey part number"
-F 7 "yes" H 6500 2150 50  0001 L CNN "is connector"
-F 8 "yes" H 6500 2250 50  0001 L CNN "is male"
-F 9 "yes" H 6500 2350 50  0001 L CNN "lead free"
-F 10 "dc1b81f16b5cdc84" H 6500 2450 50  0001 L CNN "library id"
-F 11 "Molex" H 6500 2550 50  0001 L CNN "manufacturer"
-F 12 "538-76825-0006" H 6500 2650 50  0001 L CNN "mouser part number"
-F 13 "HDR6" H 6500 2750 50  0001 L CNN "package"
-F 14 "yes" H 6500 2850 50  0001 L CNN "rohs"
-F 15 "+105°C" H 6500 2950 50  0001 L CNN "temperature range high"
-F 16 "-40°C" H 6500 3050 50  0001 L CNN "temperature range low"
-	1    6500 1150
-	1    0    0    -1
-$EndComp
-Text Label 6400 1150 0    50   ~ 0
-12V_in
-$Comp
-L power:GND #PWR0127
-U 1 1 5FE0FF44
-P 6400 2150
-F 0 "#PWR0127" H 6400 1900 50  0001 C CNN
-F 1 "GND" V 6405 1977 50  0000 C CNN
-F 2 "" H 6400 2150 50  0001 C CNN
-F 3 "" H 6400 2150 50  0001 C CNN
-	1    6400 2150
-	0    -1   -1   0
-$EndComp
-Text Label 6400 1350 0    50   ~ 0
-12V_in
-Text Label 6400 1550 0    50   ~ 0
-12V_in
-$Comp
-L power:GND #PWR0128
-U 1 1 5FFCB6FA
-P 6400 1750
-F 0 "#PWR0128" H 6400 1500 50  0001 C CNN
-F 1 "GND" V 6405 1622 50  0000 R CNN
-F 2 "" H 6400 1750 50  0001 C CNN
-F 3 "" H 6400 1750 50  0001 C CNN
-	1    6400 1750
-	0    -1   -1   0
-$EndComp
-$Comp
-L power:GND #PWR0129
-U 1 1 5FFCC514
-P 6400 1950
-F 0 "#PWR0129" H 6400 1700 50  0001 C CNN
-F 1 "GND" V 6405 1822 50  0000 R CNN
-F 2 "" H 6400 1950 50  0001 C CNN
-F 3 "" H 6400 1950 50  0001 C CNN
-	1    6400 1950
-	0    -1   -1   0
 $EndComp
 $Comp
@@
 F 0 "J8" H 3580 8992 50  0000 L CNN
 F 1 "Conn_01x06" H 3580 8901 50  0000 L CNN
-F 2 "Connector_Molex:Molex_KK-254_AE-6410-06A_1x06_P2.54mm_Vertical" H 3500 9000 50  0001 C CNN
+F 2 "Connector_Molex:Molex_Micro-Fit_3.0_43045-0612_2x03_P3.00mm_Vertical" H 3500 9000 50  0001 C CNN
 F 3 "~" H 3500 9000 50  0001 C CNN
 	1    3500 9000
@@
 Text Label 3300 8800 2    50   ~ 0
 12V
-Text Label 3300 8900 2    50   ~ 0
+Text Label 3300 9100 2    50   ~ 0
 12V
 $Comp
 L power:GND #PWR0110
 U 1 1 609B61A4
-P 3300 9000
-F 0 "#PWR0110" H 3300 8750 50  0001 C CNN
-F 1 "GND" V 3305 8872 50  0000 R CNN
-F 2 "" H 3300 9000 50  0001 C CNN
-F 3 "" H 3300 9000 50  0001 C CNN
-	1    3300 9000
+P 3300 8900
+F 0 "#PWR0110" H 3300 8650 50  0001 C CNN
+F 1 "GND" V 3305 8772 50  0000 R CNN
+F 2 "" H 3300 8900 50  0001 C CNN
+F 3 "" H 3300 8900 50  0001 C CNN
+	1    3300 8900
 	0    1    1    0
 $EndComp
@@
 L power:GND #PWR0111
 U 1 1 609B6CE7
-P 3300 9100
-F 0 "#PWR0111" H 3300 8850 50  0001 C CNN
-F 1 "GND" V 3305 8972 50  0000 R CNN
-F 2 "" H 3300 9100 50  0001 C CNN
-F 3 "" H 3300 9100 50  0001 C CNN
-	1    3300 9100
-	0    1    1    0
-$EndComp
-Text Label 3300 9200 2    50   ~ 0
+P 3300 9200
+F 0 "#PWR0111" H 3300 8950 50  0001 C CNN
+F 1 "GND" V 3305 9072 50  0000 R CNN
+F 2 "" H 3300 9200 50  0001 C CNN
+F 3 "" H 3300 9200 50  0001 C CNN
+	1    3300 9200
+	0    1    1    0
+$EndComp
+Text Label 3300 9000 2    50   ~ 0
 5V
 Text Label 3300 9300 2    50   ~ 0
@@
 Text Label 7500 7900 0    50   ~ 0
 5V
+$Comp
+L Connector_Generic:Conn_01x02 J6
+U 1 1 60A074F0
+P 7050 2300
+F 0 "J6" H 6968 1975 50  0000 C CNN
+F 1 "Conn_01x02" H 6968 2066 50  0000 C CNN
+F 2 "Connector_Molex:Molex_Mega-Fit_76829-0002_2x01_P5.70mm_Vertical" H 7050 2300 50  0001 C CNN
+F 3 "~" H 7050 2300 50  0001 C CNN
+	1    7050 2300
+	-1   0    0    1
+$EndComp
+Text Label 7250 2200 0    50   ~ 0
+12V_in
+$Comp
+L power:GND #PWR0117
+U 1 1 60A091A9
+P 7250 2300
+F 0 "#PWR0117" H 7250 2050 50  0001 C CNN
+F 1 "GND" H 7255 2127 50  0000 C CNN
+F 2 "" H 7250 2300 50  0001 C CNN
+F 3 "" H 7250 2300 50  0001 C CNN
+	1    7250 2300
+	1    0    0    -1
+$EndComp
 $EndSCHEMATC

Commit message: Add files via upload
Parts:
- removed R10: 5, Resistor_SMD:R_0402_1005Metric, symbol Device:R
- removed R23: 5k, Resistor_SMD:R_0402_1005Metric, symbol Device:R_Small
- added R11: 5, Resistor_SMD:R_0402_1005Metric, symbol Device:R
- added U6: LM317_3PinPackage, Package_TO_SOT_SMD:SOT-223-3_TabPin2, symbol Regulator_Linear:LM317_3PinPackage
Connections:
- net VCCD is gone; now on net 5V: J1.8 (Pin_8)
- net 12V: now also U6.3 (VI)
- net LASER1_CONTROL: now also Q6.1 (B)
- net LASER1_OUT: now also R11.1, U6.1 (ADJ)
- new net: R11.2, U6.2 (VO)
Other:
- moved on the sheet: D8, J2, J5
Changed lines of the file:
@@
 Text Label 6450 6400 0    50   ~ 0
 VPELT
-Text Label 7100 3350 2    50   ~ 0
-5V
-$Comp
-L Device:R R10
-U 1 1 5FBF3293
-P 7100 3500
-F 0 "R10" V 6893 3500 50  0000 C CNN
-F 1 "5" V 6984 3500 50  0000 C CNN
-F 2 "Resistor_SMD:R_0402_1005Metric" V 7030 3500 50  0001 C CNN
-F 3 "~" H 7100 3500 50  0001 C CNN
-	1    7100 3500
-	-1   0    0    1
-$EndComp
-Text Label 7250 3650 0    50   ~ 0
-LASER1_OUT
-Text Label 6600 4100 2    50   ~ 0
-LASER1_CONTROL
 Wire Notes Line
 	8950 3000 5850 3000
-$Comp
-L Connector_Generic:Conn_01x02 J2
-U 1 1 5FDBBF57
-P 8500 3650
-F 0 "J2" H 8580 3642 50  0000 L CNN
-F 1 "Laser 1" H 8580 3551 50  0000 L CNN
-F 2 "MJ1-2533-SMT:CUI_MJ1-2533-SMT" H 8500 3650 50  0001 C CNN
-F 3 "~" H 8500 3650 50  0001 C CNN
-	1    8500 3650
-	1    0    0    -1
-$EndComp
-Wire Wire Line
-	7250 3750 7100 3750
-Wire Wire Line
-	7100 3750 7100 3900
-Text Label 8300 3750 2    50   ~ 0
-LASER1_OUT
 Wire Notes Line
 	5850 4750 8950 4750
@@
 Wire Notes Line
 	8950 3000 8950 4750
-$Comp
-L Device:R_Small R23
-U 1 1 5FF85ED9
-P 6700 4100
-F 0 "R23" V 6504 4100 50  0000 C CNN
-F 1 "5k" V 6595 4100 50  0000 C CNN
-F 2 "Resistor_SMD:R_0402_1005Metric" H 6700 4100 50  0001 C CNN
-F 3 "~" H 6700 4100 50  0001 C CNN
-	1    6700 4100
-	0    -1   -1   0
-$EndComp
 $Comp
 L Driver_Motor:DRV8834 U9
@@
 L Connector_Generic:Conn_01x02 J5
 U 1 1 60901E57
-P 10050 3050
-F 0 "J5" H 10130 3042 50  0000 L CNN
-F 1 "Conn_01x02" H 10130 2951 50  0000 L CNN
-F 2 "Connector_Molex:Molex_KK-254_AE-6410-02A_1x02_P2.54mm_Vertical" H 10050 3050 50  0001 C CNN
-F 3 "~" H 10050 3050 50  0001 C CNN
-	1    10050 3050
-	1    0    0    -1
-$EndComp
-Text Label 9850 3050 2    50   ~ 0
+P 10700 2750
+F 0 "J5" H 10780 2742 50  0000 L CNN
+F 1 "Conn_01x02" H 10780 2651 50  0000 L CNN
+F 2 "Connector_Molex:Molex_KK-254_AE-6410-02A_1x02_P2.54mm_Vertical" H 10700 2750 50  0001 C CNN
+F 3 "~" H 10700 2750 50  0001 C CNN
+	1    10700 2750
+	1    0    0    -1
+$EndComp
+Text Label 10500 2750 2    50   ~ 0
 12V
-Text Label 9850 3150 2    50   ~ 0
+Text Label 10500 2850 2    50   ~ 0
 SOLENOID_GND
 $Comp
 L Device:D D8
 U 1 1 609046FF
-P 10100 4600
-F 0 "D8" H 10100 4384 50  0000 C CNN
-F 1 "CMPD914E" H 10100 4475 50  0000 C CNN
-F 2 "Package_TO_SOT_SMD:SOT-23" H 10100 4600 50  0001 C CNN
-F 3 "~" H 10100 4600 50  0001 C CNN
-	1    10100 4600
-	-1   0    0    1
-$EndComp
-Text Label 9950 4600 2    50   ~ 0
+P 9800 2800
+F 0 "D8" H 9800 2584 50  0000 C CNN
+F 1 "CMPD914E" H 9800 2675 50  0000 C CNN
+F 2 "Package_TO_SOT_SMD:SOT-23" H 9800 2800 50  0001 C CNN
+F 3 "~" H 9800 2800 50  0001 C CNN
+	1    9800 2800
+	0    1    1    0
+$EndComp
+Text Label 9800 2950 2    50   ~ 0
 SOLENOID_GND
-Text Label 10250 4600 0    50   ~ 0
+Text Label 9800 2650 1    50   ~ 0
 12V
 $Comp
@@
 	1    2300 5500
 	0    1    1    0
-$EndComp
-$Comp
-L Device:Q_NPN_BCE Q6
-U 1 1 60956273
-P 7000 4100
-F 0 "Q6" H 7190 4146 50  0000 L CNN
-F 1 "FMMT634Q" H 7190 4055 50  0000 L CNN
-F 2 "Package_TO_SOT_SMD:SOT-23" H 7200 4200 50  0001 C CNN
-F 3 "~" H 7000 4100 50  0001 C CNN
-	1    7000 4100
-	1    0    0    -1
-$EndComp
-$Comp
-L power:GND #PWR0121
-U 1 1 609573A3
-P 7100 4300
-F 0 "#PWR0121" H 7100 4050 50  0001 C CNN
-F 1 "GND" H 7105 4127 50  0000 C CNN
-F 2 "" H 7100 4300 50  0001 C CNN
-F 3 "" H 7100 4300 50  0001 C CNN
-	1    7100 4300
-	1    0    0    -1
 $EndComp
 $Comp
@@
 Text Label 10250 6550 0    50   ~ 0
 LED_GND
-Text Label 8300 3650 2    50   ~ 0
-LASER1_GND
-Wire Wire Line
-	7250 3650 7100 3650
-Text Label 7250 3750 0    50   ~ 0
-LASER1_GND
 Text Label 6450 6500 0    50   ~ 0
 PELT_GND
@@
 	1    0    0    -1
 $EndComp
+Text Label 7100 5550 2    50   ~ 0
+VCCD
+Text Label 7250 5550 0    50   ~ 0
+5V
+Wire Wire Line
+	7250 5550 7100 5550
+Text Label 10850 5500 0    50   ~ 0
+LASER1_OUT
+$Comp
+L power:GND #PWR0118
+U 1 1 60B6BDCF
+P 7700 4100
+F 0 "#PWR0118" H 7700 3850 50  0001 C CNN
+F 1 "GND" H 7705 3927 50  0000 C CNN
+F 2 "" H 7700 4100 50  0001 C CNN
+F 3 "" H 7700 4100 50  0001 C CNN
+	1    7700 4100
+	1    0    0    -1
+$EndComp
+Wire Wire Line
+	7700 3700 7700 3450
+Wire Wire Line
+	7300 3350 7700 3350
+Text Label 7400 3900 2    50   ~ 0
+LASER1_CONTROL
+Wire Wire Line
+	7300 3350 7200 3350
+Connection ~ 7300 3350
+Wire Wire Line
+	6450 3750 6450 3650
+Wire Wire Line
+	7300 3750 6450 3750
+Wire Wire Line
+	7300 3350 7300 3750
+Wire Wire Line
+	6750 3350 6900 3350
+$Comp
+L Device:R R11
+U 1 1 60B09DCA
+P 7050 3350
+F 0 "R11" V 6843 3350 50  0000 C CNN
+F 1 "5" V 6934 3350 50  0000 C CNN
+F 2 "Resistor_SMD:R_0402_1005Metric" V 6980 3350 50  0001 C CNN
+F 3 "~" H 7050 3350 50  0001 C CNN
+	1    7050 3350
+	0    1    1    0
+$EndComp
+Text Label 6150 3350 2    50   ~ 0
+12V
+$Comp
+L Regulator_Linear:LM317_3PinPackage U6
+U 1 1 60B07CEE
+P 6450 3350
+F 0 "U6" H 6450 3592 50  0000 C CNN
+F 1 "LM317_3PinPackage" H 6450 3501 50  0000 C CNN
+F 2 "Package_TO_SOT_SMD:SOT-223-3_TabPin2" H 6450 3600 50  0001 C CIN
+F 3 "http://www.ti.com/lit/ds/symlink/lm317.pdf" H 6450 3350 50  0001 C CNN
+	1    6450 3350
+	1    0    0    -1
+$EndComp
+Text Label 6550 4350 2    50   ~ 0
+LASER1_GND
+Text Label 6550 4450 2    50   ~ 0
+LASER1_OUT
+$Comp
+L Connector_Generic:Conn_01x02 J2
+U 1 1 5FDBBF57
+P 6750 4350
+F 0 "J2" H 6830 4342 50  0000 L CNN
+F 1 "Laser 1" H 6830 4251 50  0000 L CNN
+F 2 "MJ1-2533-SMT:CUI_MJ1-2533-SMT" H 6750 4350 50  0001 C CNN
+F 3 "~" H 6750 4350 50  0001 C CNN
+	1    6750 4350
+	1    0    0    -1
+$EndComp
+$Comp
+L Device:Q_NPN_BCE Q6
+U 1 1 60B1620C
+P 7600 3900
+F 0 "Q6" H 7790 3946 50  0000 L CNN
+F 1 "FMMT634Q" H 7790 3855 50  0000 L CNN
+F 2 "Package_TO_SOT_SMD:SOT-23" H 7800 4000 50  0001 C CNN
+F 3 "~" H 7600 3900 50  0001 C CNN
+	1    7600 3900
+	1    0    0    -1
+$EndComp
+Text Label 7700 3350 0    50   ~ 0
+LASER1_OUT
+Text Label 7700 3450 0    50   ~ 0
+LASER1_GND
 $EndSCHEMATC
